File: hardware/cv-strip.brd (EAGLE design)
At the start: 140.7 x 40.8 mm, 83 parts, among them IC1 PIC16F1825SO14, IC2 74HC595D, IC3 MCP4728_QUAD_DAC, IC4 LM324D, IC5 REG1117, IC6 74HC595D

Commit message: getting there
Parts:
- removed JP1: (no value), pinhead:1X02
- added U$2: PWR_SOCKET_2_1MM, jason_eagle6:PWR_SOCKET_2_1MM
- moved C24 27.9 mm to (149.4, 13.0), turned to 270 degrees
- moved R34 23.6 mm to (140.3, 13.0)
- moved DRM8 22.9 mm to (144.8, 8.89)
- moved C1 18.0 mm to (79.4, 25.7), turned to 270 degrees
- moved C19 18.0 mm to (149.2, 25.7), turned to 270 degrees
- moved C4 17.9 mm to (79.2, 13.1), turned to 270 degrees
- moved C2 16.8 mm to (66.7, 25.8), turned to 270 degrees
- moved C3 16.8 mm to (66.7, 13.1), turned to 270 degrees
- moved C16 16.7 mm to (136.5, 25.7), turned to 270 degrees
- moved C15 15.5 mm to (123.8, 25.7), turned to 270 degrees
- moved C17 14.4 mm to (87.1, 29.7), turned to 0 degrees
- moved C21 14.4 mm to (111.1, 25.7), turned to 270 degrees
- moved C23 14.3 mm to (123.8, 12.8), turned to 270 degrees
- moved C20 14.3 mm to (111.1, 12.8), turned to 270 degrees
- moved R24 14.1 mm to (140.3, 25.7)
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Connections:
- net GND: now also U$2.PIN; no longer JP1.1
- net N$40: now also U$2.BARREL; no longer JP1.2
- net VOUTA: now also IC4.5; no longer IC4.10
- net VOUTB: now also IC4.3; no longer IC4.12
- net VOUTC: now also IC4.12; no longer IC4.3
- net VOUTD: now also IC4.10; no longer IC4.5
Routing:
- net N$40: track 4.32 -> 48.9 mm
- net N$48: track 29.7 -> 59.7 mm
- net N$46: track 16.9 -> 46.1 mm, vias 0 -> 2
- net N$47: track 45.2 -> 73.4 mm
- net N$15: track 10.2 -> 34.5 mm, vias 0 -> 2
- net N$53: track 30.5 -> 53.7 mm, vias 2 -> 0
- net N$16: track 28.5 -> 45.9 mm
- net SR_DAT2: track 26.7 -> 43.9 mm
- net VDD: track 217.3 -> 232.1 mm, vias 9 -> 7
- net N$22: track 36.2 -> 50.1 mm, vias 2 -> 3
- net N$21: track 36.2 -> 49.7 mm, vias 0 -> 3
- net N$13: track 20.9 -> 34.2 mm, vias 2 -> 0
- net SR_CLK: track 41.2 -> 28.0 mm, vias 2 -> 3
- net VOUTA: track 22.2 -> 10.6 mm
- net N$12: track 11.8 -> 22.9 mm, vias 0 -> 2
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- removed copper zone on layer 1, net GND
Other:
- board size 140.7 x 40.8 mm -> 152.5 x 43.6 mm

Commit message: almost done?
Parts:
- removed C22, C24: (no value), rcl:C0805
- removed R31, R32, R33: (no value), rcl:R0805
- added C10, C13: (no value), rcl:C0805
- added R15, R16, R6: (no value), rcl:R0805
- C11, C5: device resistor:E2,5-5 -> rcl:C0805
- C20, C21: device rcl:C0805 -> resistor:E2,5-5
- IC3: value MCP4728_QUAD_DAC -> 74HC595D; device jason_eagle6:MSOP10 -> 74xx-eu:SO16
- IC4: value LM324D -> MCP4728_QUAD_DAC; device linear:SO14 -> jason_eagle6:MSOP10
- IC5: value REG1117 -> LM324D; device burr-brown:SOT223 -> linear:SO14
- IC6: value 74HC595D -> REG1117; device 74xx-eu:SO16 -> burr-brown:SOT223
- moved R10 99.0 mm to (127.6, 13.0), turned to 90 degrees
- moved R24 97.9 mm to (43.2, 38.1), turned to 0 degrees
- moved C19 92.3 mm to (57.0, 29.5), turned to 0 degrees
- moved R7 91.7 mm to (114.9, 25.7), turned to 90 degrees
- moved R29 82.1 mm to (24.1, 38.1), turned to 270 degrees
- moved C5 79.8 mm to (149.4, 13.0), flipped to the bottom
- moved C6 78.0 mm to (136.5, 13.0), turned to 270 degrees
- moved R17 71.9 mm to (57.1, 40.6), turned to 0 degrees
- moved R14 71.5 mm to (57.8, 25.8), turned to 90 degrees
- moved R8 71.4 mm to (102.2, 25.7)
- moved C2 69.9 mm to (136.5, 25.7)
- moved C1 69.8 mm to (149.2, 25.7)
- moved R2 65.3 mm to (122.8, 31.8), turned to 0 degrees
- moved R3 61.5 mm to (116.2, 31.8), turned to 0 degrees
- moved R1 58.9 mm to (129.0, 31.6), turned to 0 degrees
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- renumbered ACT to L1, C23 to C7, D3 to D2, DRMA to DRM1, GATA to CLK2, OK1 to IC7, PWR to L3, R30 to R11, R34 to R9, STS to L2, SYNC1 to CLK1, U$1 to D1
Connections:
- net GND: now also C10.1, C11.1, C12.2, C13.2, C17.2, C18.2, C19.1, C20.-, C21.-, C5.2, IC3.13, IC3.8, IC4.10, IC4.4, IC5.11, IC6.1, R1.2, R18.1, R19.1, R2.2, R24.1, R28.2, R3.2; no longer C11.-, C12.1, C17.1, C18.1, C19.2, C20.2, C21.2, C22.2, C24.2, C5.-, IC3.10, IC3.4, IC4.11, IC5.1, IC6.13, IC6.8, R10.2, R12.2, R13.2, R14.2, R20.1, R23.1, R28.1
- net MIDI_IN: now also R27.1; no longer R8.1
- net N$1: now also C16.1, R15.2; no longer C4.1, R4.2
- net N$12: now also IC3.15, R15.1; no longer IC2.15, R4.1
- net N$13: now also IC3.1, R16.1; no longer IC2.1, R3.1
- net N$15: now also IC3.3, R13.1; no longer IC2.3, R1.1
- net N$16: now also IC3.2, R14.1; no longer IC2.2, R2.1
- net N$2: now also IC5.1, R17.2; no longer IC4.1, R27.2
- net N$20: now also C4.1, R8.2; no longer C21.1, R32.2
- net N$21: now also IC4.2, R22.2; no longer IC3.2, R19.2
- net N$22: now also IC4.3, R21.2; no longer IC3.3, R18.2
- net N$23: now also C3.1, R7.2; no longer C15.1, R33.2
- net N$24: now also C2.1, R6.2; no longer C16.1, R17.2
- net N$25: now also IC5.2, R17.1, R18.2; no longer IC4.2, R27.1, R28.2
- net N$26: now also IC5.6, R19.2, R20.1; no longer IC4.6, R22.1, R23.2
- net N$27: now also IC5.9, R25.2, R26.1; no longer IC4.9, R20.2, R21.1
- net N$28: now also IC5.13, R23.1, R24.2; no longer IC4.13, R25.2, R26.1
- net N$29: now also R29.1; no longer R7.1
- net N$3: now also IC5.7, R20.2; no longer IC4.7, R22.2
- net N$30: now also R29.2; no longer R7.2
- net N$32: now also C1.1, R5.2; no longer C19.1, R24.2
- net N$33: now also C8.1, R12.2; no longer C20.1, R29.2
- net N$35: now also R1.1; no longer R14.1
- net N$36: now also R3.1; no longer R13.1
- net N$37: now also R2.1; no longer R12.1
- net N$4: now also IC5.8, R26.2; no longer IC4.8, R21.2
- net N$41: now also C6.1, R10.2; no longer C22.1, R31.2
- net N$42: now also R28.1; no longer R10.1
- net N$43: now also IC2.15, R8.1; no longer IC6.15, R32.1
- net N$46: now also IC2.1, R7.1; no longer IC6.1, R33.1
- net N$47: now also IC2.3, R5.1; no longer IC6.3, R24.1
- net N$48: now also IC2.2, R6.1; no longer IC6.2, R17.1
- net N$49: now also IC2.5; no longer IC6.5
- net N$5: now also IC5.14, R23.2; no longer IC4.14, R26.2
- net N$50: now also IC2.6, R10.1; no longer IC6.6, R31.1
- net N$51: now also IC2.4, R12.1; no longer IC6.4, R29.1
- net N$52: now also C5.1; no longer C24.1
- net N$53: now also IC2.7; no longer IC6.7
- net N$6: now also C17.1, R16.2; no longer C3.1, R3.2
- net N$7: now also C15.1, R14.2; no longer C2.1, R2.2
- net N$8: now also C14.1, R13.2; no longer C1.1, R1.2
- net N$9: now also R4.2; no longer R5.2
- net SR_CLK: now also IC3.11; no longer IC6.11
- net SR_DAT: now also IC3.14; no longer IC2.14
- net SR_DAT2: now also IC2.14; no longer IC6.14
- net SR_RCK: now also IC3.12; no longer IC6.12
- net VDD: now also C11.2, C12.1, C13.1, C19.2, C20.+, IC3.10, IC3.16, IC4.1, IC6.2, R21.1, R22.1, R27.2, R4.1; no longer C12.2, C14.1, C17.2, C5.+, C8.1, IC3.1, IC5.2, IC6.10, IC6.16, R18.1, R19.1, R5.1, R8.2
- net VIN: now also C10.2, C18.1, C21.+, IC5.4, IC6.3; no longer C11.+, C18.2, C6.1, IC4.4, IC5.3
- net VOUTA: now also IC4.6, IC5.5; no longer IC3.6, IC4.5
- net VOUTB: now also IC4.7, IC5.3; no longer IC3.7, IC4.3
- net VOUTC: now also IC4.8, IC5.12; no longer IC3.8, IC4.12
- net VOUTD: now also IC4.9, IC5.10; no longer IC3.9, IC4.10
Routing:
- net N$22: track 50.1 -> 50.9 mm
- net STATUS_LED: track 47.0 -> 46.4 mm
- net N$3: track 13.0 -> 13.1 mm, vias 0 -> 1
- net GND: vias 0 -> 3
- added copper zone on layer 1, net GND
Other:
- outline, holes or cut-outs redrawn
- board text added: "converter"
- board text added: "hotchk155"
- board text added: "midi-to-cv"
- board text added: "rev 1"

Commit message: tweaks
Parts:
- renumbered ISCP to ICSP
Changed lines of the file:
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@@
 <attribute name="VALUE" x="81.788" y="14.351" size="1.27" layer="28" rot="MR270"/>
 </element>
-<element name="ISCP" library="tag-connect" package="TC2030-MCP-NL" value="" x="84.709" y="26.67" smashed="yes" rot="MR270">
-<attribute name="NAME" x="83.439" y="27.305" size="1.27" layer="26" rot="MR270"/>
+<element name="ICSP" library="tag-connect" package="TC2030-MCP-NL" value="" x="84.709" y="26.67" smashed="yes" rot="MR270">
+<attribute name="NAME" x="82.677" y="20.066" size="1.27" layer="26" rot="MR180"/>
 </element>
 <element name="L3" library="led" package="LED3MM" value="" x="128.905" y="35.687" smashed="yes" rot="R270">
@@
 </element>
 <element name="DRM1" library="jason_eagle6" package="VERTICAL_3_5MM_SOCKET" value="VERTICAL_3_5MM_SOCKET" x="106.68" y="21.59" smashed="yes">
-<attribute name="NAME" x="104.267" y="27.686" size="1.27" layer="21"/>
+<attribute name="NAME" x="104.394" y="27.813" size="1.27" layer="21"/>
 </element>
 <element name="DRM2" library="jason_eagle6" package="VERTICAL_3_5MM_SOCKET" value="VERTICAL_3_5MM_SOCKET" x="119.38" y="21.59" smashed="yes">
-<attribute name="NAME" x="116.967" y="27.432" size="1.27" layer="21"/>
+<attribute name="NAME" x="116.967" y="27.813" size="1.27" layer="21"/>
 </element>
 <element name="DRM3" library="jason_eagle6" package="VERTICAL_3_5MM_SOCKET" value="VERTICAL_3_5MM_SOCKET" x="132.08" y="21.59" smashed="yes">
-<attribute name="NAME" x="129.54" y="27.559" size="1.27" layer="21"/>
+<attribute name="NAME" x="129.54" y="27.813" size="1.27" layer="21"/>
 </element>
 <element name="DRM4" library="jason_eagle6" package="VERTICAL_3_5MM_SOCKET" value="VERTICAL_3_5MM_SOCKET" x="144.78" y="21.59" smashed="yes">
-<attribute name="NAME" x="142.494" y="27.432" size="1.27" layer="21"/>
+<attribute name="NAME" x="142.494" y="27.813" size="1.27" layer="21"/>
 </element>
 <element name="DRM5" library="jason_eagle6" package="VERTICAL_3_5MM_SOCKET" value="VERTICAL_3_5MM_SOCKET" x="106.68" y="8.89" smashed="yes">
@@
 <contactref element="C15" pad="2"/>
 <contactref element="C14" pad="2"/>
-<contactref element="ISCP" pad="3"/>
+<contactref element="ICSP" pad="3"/>
 <contactref element="IC4" pad="4"/>
 <contactref element="R1" pad="2"/>
@@
 <contactref element="IC3" pad="14"/>
 <contactref element="IC1" pad="13"/>
-<contactref element="ISCP" pad="4"/>
+<contactref element="ICSP" pad="4"/>
 <wire x1="90.11" y1="24.13" x2="88.265" y2="24.13" width="0.3048" layer="16"/>
 <via x="88.265" y="24.13" extent="1-16" drill="0.6"/>
@@
 <signal name="N$34">
 <contactref element="IC1" pad="4"/>
-<contactref element="ISCP" pad="1"/>
+<contactref element="ICSP" pad="1"/>
 <wire x1="85.344" y1="25.4" x2="86.36" y2="25.4" width="0.3048" layer="16"/>
 <via x="86.36" y="25.4" extent="1-16" drill="0.6"/>
@@
 <contactref element="IC1" pad="1"/>
 <contactref element="C19" pad="2"/>
-<contactref element="ISCP" pad="2"/>
+<contactref element="ICSP" pad="2"/>
 <contactref element="IC7" pad="8"/>
 <contactref element="R27" pad="2"/>
@@
 <wire x1="60.775409375" y1="32.708409375" x2="59.42" y2="31.353" width="0.4064" layer="16"/>
 <wire x1="63.5" y1="33.97" x2="66.04" y2="33.97" width="0.4064" layer="16"/>
-<wire x1="52.2781" y1="31.353" x2="56.007" y2="31.353" width="0.4064" layer="16"/>
 <wire x1="56.007" y1="31.353" x2="59.42" y2="31.353" width="0.4064" layer="16"/>
 <wire x1="56.073" y1="29.464" x2="56.073" y2="31.287" width="0.4064" layer="16"/>
@@
 <wire x1="58.477590625" y1="32.708409375" x2="57.15" y2="34.036" width="0.8128" layer="1"/>
 <wire x1="57.15" y1="34.036" x2="57.15" y2="41.275" width="0.8128" layer="1"/>
+<wire x1="52.2781" y1="31.353" x2="56.007" y2="31.353" width="0.3048" layer="16"/>
 </signal>
 <signal name="VIN">
@@
 <contactref element="IC2" pad="14"/>
 <contactref element="IC1" pad="12"/>
-<contactref element="ISCP" pad="5"/>
+<contactref element="ICSP" pad="5"/>
 <wire x1="90.11" y1="22.86" x2="85.344" y2="22.86" width="0.3048" layer="16"/>
 <via x="96.52" y="1.27" extent="1-16" drill="0.6"/>

Commit message: pcb v1
Changed lines of the file:
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@@
 <layer number="27" name="tValues" color="7" fill="1" visible="yes" active="yes"/>
 <layer number="28" name="bValues" color="7" fill="1" visible="yes" active="yes"/>
-<layer number="29" name="tStop" color="7" fill="3" visible="no" active="yes"/>
-<layer number="30" name="bStop" color="7" fill="6" visible="no" active="yes"/>
-<layer number="31" name="tCream" color="7" fill="4" visible="no" active="yes"/>
-<layer number="32" name="bCream" color="7" fill="5" visible="no" active="yes"/>
-<layer number="33" name="tFinish" color="6" fill="3" visible="no" active="yes"/>
-<layer number="34" name="bFinish" color="6" fill="6" visible="no" active="yes"/>
-<layer number="35" name="tGlue" color="7" fill="4" visible="no" active="yes"/>
-<layer number="36" name="bGlue" color="7" fill="5" visible="no" active="yes"/>
-<layer number="37" name="tTest" color="7" fill="1" visible="no" active="yes"/>
-<layer number="38" name="bTest" color="7" fill="1" visible="no" active="yes"/>
+<layer number="29" name="tStop" color="7" fill="3" visible="yes" active="yes"/>
+<layer number="30" name="bStop" color="7" fill="6" visible="yes" active="yes"/>
+<layer number="31" name="tCream" color="7" fill="4" visible="yes" active="yes"/>
+<layer number="32" name="bCream" color="7" fill="5" visible="yes" active="yes"/>
+<layer number="33" name="tFinish" color="6" fill="3" visible="yes" active="yes"/>
+<layer number="34" name="bFinish" color="6" fill="6" visible="yes" active="yes"/>
+<layer number="35" name="tGlue" color="7" fill="4" visible="yes" active="yes"/>
+<layer number="36" name="bGlue" color="7" fill="5" visible="yes" active="yes"/>
+<layer number="37" name="tTest" color="7" fill="1" visible="yes" active="yes"/>
+<layer number="38" name="bTest" color="7" fill="1" visible="yes" active="yes"/>
 <layer number="39" name="tKeepout" color="4" fill="11" visible="yes" active="yes"/>
 <layer number="40" name="bKeepout" color="1" fill="11" visible="yes" active="yes"/>
@@
 <layer number="42" name="bRestrict" color="1" fill="10" visible="yes" active="yes"/>
 <layer number="43" name="vRestrict" color="2" fill="10" visible="yes" active="yes"/>
-<layer number="44" name="Drills" color="7" fill="1" visible="no" active="yes"/>
+<layer number="44" name="Drills" color="7" fill="1" visible="yes" active="yes"/>
 <layer number="45" name="Holes" color="7" fill="1" visible="yes" active="yes"/>
-<layer number="46" name="Milling" color="3" fill="1" visible="no" active="yes"/>
-<layer number="47" name="Measures" color="7" fill="1" visible="no" active="yes"/>
+<layer number="46" name="Milling" color="3" fill="1" visible="yes" active="yes"/>
+<layer number="47" name="Measures" color="7" fill="1" visible="yes" active="yes"/>
 <layer number="48" name="Document" color="7" fill="1" visible="yes" active="yes"/>
 <layer number="49" name="Reference" color="7" fill="1" visible="yes" active="yes"/>
 <layer number="50" name="dxf" color="7" fill="1" visible="no" active="no"/>
-<layer number="51" name="tDocu" color="7" fill="1" visible="no" active="yes"/>
+<layer number="51" name="tDocu" color="7" fill="1" visible="yes" active="yes"/>
 <layer number="52" name="bDocu" color="7" fill="1" visible="yes" active="yes"/>
 <layer number="53" name="tGND_GNDA" color="7" fill="9" visible="no" active="no"/>
@@
 <layer number="103" name="tMap" color="7" fill="1" visible="yes" active="yes"/>
 <layer number="104" name="Name" color="7" fill="1" visible="yes" active="yes"/>
-<layer number="105" name="tPlate" color="7" fill="1" visible="no" active="yes"/>
-<layer number="106" name="bPlate" color="7" fill="1" visible="no" active="yes"/>
+<layer number="105" name="tPlate" color="7" fill="1" visible="yes" active="yes"/>
+<layer number="106" name="bPlate" color="7" fill="1" visible="yes" active="yes"/>
 <layer number="107" name="Crop" color="7" fill="1" visible="yes" active="yes"/>
 <layer number="108" name="fp8" color="7" fill="1" visible="yes" active="yes"/>
@@
 <text x="57.531" y="30.607" size="2.032" layer="25" font="vector">rev 1</text>
 <text x="30.734" y="7.366" size="2.032" layer="25" font="vector" rot="R90">hotchk155</text>
+<hole x="90.678" y="31.678" drill="3.2"/>
 </plain>
 <attributes>
@@
 </element>
 <element name="C9" library="rcl" package="C0805" value="" x="87.122" y="29.718" smashed="yes" rot="MR0">
-<attribute name="NAME" x="89.789" y="31.115" size="1.27" layer="26" rot="MR0"/>
+<attribute name="NAME" x="88.773" y="27.178" size="1.27" layer="26" rot="MR0"/>
 <attribute name="VALUE" x="88.392" y="27.178" size="1.27" layer="28" rot="MR0"/>
 </element>
@@
 </element>
 <element name="C11" library="rcl" package="C0805" value="" x="92.71" y="27.559" smashed="yes" rot="MR180">
-<attribute name="NAME" x="90.424" y="30.099" size="1.27" layer="26" rot="MR180"/>
+<attribute name="NAME" x="94.869" y="28.321" size="1.27" layer="26" rot="MR180"/>
 <attribute name="VALUE" x="91.44" y="30.099" size="1.27" layer="28" rot="MR180"/>
 </element>
 <element name="D2" library="jasons_stuff" package="DO-VERT" value="1N4004" x="88.9" y="36.83" smashed="yes" rot="R90">
-<attribute name="NAME" x="90.043" y="34.417" size="1.27" layer="25" ratio="10" rot="R180"/>
+<attribute name="NAME" x="88.011" y="34.798" size="1.27" layer="25" ratio="10" rot="R180"/>
 </element>
 <element name="MIDI_IN" library="jason_eagle6" package="EDGEDIN" value="DIN5PIN" x="16.51" y="35.052" smashed="yes">
@@
 <contactref element="IC3" pad="1"/>
 <contactref element="R16" pad="1"/>
-<wire x1="82.9056" y1="3.175" x2="80.137" y2="3.175" width="0.3048" layer="16"/>
-<wire x1="80.137" y1="3.175" x2="79.121" y2="2.159" width="0.3048" layer="16"/>
-<wire x1="79.121" y1="2.159" x2="59.944" y2="2.159" width="0.3048" layer="16"/>
+<wire x1="82.9056" y1="3.175" x2="77.597" y2="3.175" width="0.3048" layer="16"/>
+<wire x1="77.597" y1="3.175" x2="76.581" y2="2.159" width="0.3048" layer="16"/>
+<wire x1="76.581" y1="2.159" x2="59.944" y2="2.159" width="0.3048" layer="16"/>
 <wire x1="59.944" y1="2.159" x2="57.658" y2="4.445" width="0.3048" layer="16"/>
 <wire x1="57.658" y1="4.445" x2="57.658" y2="12.004" width="0.3048" layer="16"/>
