File: hardware/cv-strip.brd (EAGLE design)
At the start: 152.5 x 43.6 mm, 123 parts, among them IC1 LPC812, IC2 AD5696R, IC3 MC14094B, IC4 MC14094B, IC5 LM324D, IC6 REG1117, IC7 6N138, IC8 24LC_64T-I/OT, IC9 MIC5504-2.8YM5-TR

Commit message: rev3 PCB final
Connections:
- net SCL: now also IC1.9; no longer IC1.8
- net SDA: now also IC1.8; no longer IC1.9
- net STATUS_LED: now also IC1.3; no longer IC1.20
Routing:
- net STATUS_LED: track 39.4 -> 34.1 mm
- net 3V3: track 79.1 -> 80.1 mm
- net MIDI_IN: track 96.4 -> 97.4 mm
- net GT2_VSEL: track 71.8 -> 72.5 mm
Changed lines of the file:
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@@
 <wire x1="89.535" y1="28.6385" x2="91.059" y2="28.6385" width="0.3048" layer="16"/>
 <via x="91.059" y="28.6385" extent="1-16" drill="0.6"/>
-<wire x1="91.059" y1="28.6385" x2="93.0275" y2="26.67" width="0.3048" layer="1"/>
 <via x="93.0275" y="26.67" extent="1-16" drill="0.6"/>
 <wire x1="93.0275" y1="26.67" x2="91.948" y2="26.67" width="0.3048" layer="16"/>
+<wire x1="91.059" y1="28.6385" x2="92.6465" y2="28.6385" width="0.3048" layer="1"/>
+<wire x1="93.0275" y1="26.67" x2="93.0275" y2="28.2575" width="0.3048" layer="1"/>
+<wire x1="93.0275" y1="28.2575" x2="92.6465" y2="28.6385" width="0.3048" layer="1"/>
 </signal>
 <signal name="SCL">
@@
 <wire x1="50.7873" y1="31.4198" x2="50.8" y2="31.4325" width="0.3048" layer="16"/>
 <wire x1="50.8" y1="31.4325" x2="71.12" y2="31.4325" width="0.3048" layer="1"/>
-<contactref element="IC1" pad="8"/>
 <wire x1="71.12" y1="31.4325" x2="74.295" y2="31.4325" width="0.3048" layer="1"/>
 <wire x1="74.295" y1="31.4325" x2="74.7395" y2="30.988" width="0.3048" layer="1"/>
 <wire x1="74.7395" y1="30.988" x2="83.312" y2="30.988" width="0.3048" layer="1"/>
-<via x="91.7575" y="25.019" extent="1-16" drill="0.6"/>
+<via x="92.456" y="24.13" extent="1-16" drill="0.6"/>
 <wire x1="89.281" y1="25.019" x2="83.312" y2="30.988" width="0.3048" layer="1"/>
-<wire x1="94.3578" y1="25.045" x2="91.7835" y2="25.045" width="0.3048" layer="16"/>
-<wire x1="91.7835" y1="25.045" x2="91.7575" y2="25.019" width="0.3048" layer="16"/>
-<wire x1="89.281" y1="25.019" x2="91.7575" y2="25.019" width="0.3048" layer="1"/>
+<contactref element="IC1" pad="9"/>
+<wire x1="89.281" y1="25.019" x2="91.567" y2="25.019" width="0.3048" layer="1"/>
+<wire x1="94.3578" y1="24.395" x2="92.721" y2="24.395" width="0.3048" layer="16"/>
+<wire x1="92.721" y1="24.395" x2="92.456" y2="24.13" width="0.3048" layer="16"/>
+<wire x1="91.567" y1="25.019" x2="92.456" y2="24.13" width="0.3048" layer="1"/>
 </signal>
 <signal name="SDA">
@@
 <wire x1="73.66" y1="33.34" x2="73.66" y2="30.48" width="0.3048" layer="16"/>
 <via x="73.66" y="30.48" extent="1-16" drill="0.6"/>
-<contactref element="IC1" pad="9"/>
 <contactref element="IC8" pad="3"/>
 <wire x1="57.023" y1="30.48" x2="48.768" y2="30.48" width="0.3048" layer="1"/>
@@
 <wire x1="47.8282" y1="29.5402" x2="48.768" y2="30.48" width="0.3048" layer="16"/>
 <via x="48.768" y="30.48" extent="1-16" drill="0.6"/>
-<wire x1="94.3578" y1="24.395" x2="92.975" y2="24.395" width="0.3048" layer="16"/>
-<wire x1="92.975" y1="24.395" x2="92.71" y2="24.13" width="0.3048" layer="16"/>
-<via x="92.71" y="24.13" extent="1-16" drill="0.6"/>
-<wire x1="92.71" y1="24.13" x2="89.3445" y2="24.13" width="0.3048" layer="1"/>
+<via x="90.7415" y="24.13" extent="1-16" drill="0.6"/>
+<wire x1="90.7415" y1="24.13" x2="89.3445" y2="24.13" width="0.3048" layer="1"/>
 <wire x1="89.3445" y1="24.13" x2="82.9945" y2="30.48" width="0.3048" layer="1"/>
+<contactref element="IC1" pad="8"/>
+<wire x1="94.3578" y1="25.045" x2="91.6565" y2="25.045" width="0.3048" layer="16"/>
+<wire x1="91.6565" y1="25.045" x2="90.7415" y2="24.13" width="0.3048" layer="16"/>
 </signal>
 <signal name="N$2">
@@
 <wire x1="103.759" y1="33.528" x2="117.856" y2="33.528" width="0.3048" layer="1"/>
 <wire x1="117.856" y1="33.528" x2="123.825" y2="39.497" width="0.3048" layer="1"/>
-<wire x1="97.8535" y1="30.6705" x2="100.9015" y2="30.6705" width="0.3048" layer="1"/>
+<wire x1="97.9805" y1="30.6705" x2="100.9015" y2="30.6705" width="0.3048" layer="1"/>
 <wire x1="100.9015" y1="30.6705" x2="103.759" y2="33.528" width="0.3048" layer="1"/>
-<contactref element="IC1" pad="20"/>
-<wire x1="88.5222" y1="29.595" x2="89.912" y2="29.595" width="0.3048" layer="16"/>
-<wire x1="89.912" y1="29.595" x2="89.916" y2="29.591" width="0.3048" layer="16"/>
-<via x="89.916" y="29.591" extent="1-16" drill="0.6"/>
-<wire x1="89.916" y1="29.591" x2="96.774" y2="29.591" width="0.3048" layer="1"/>
-<wire x1="96.774" y1="29.591" x2="97.8535" y2="30.6705" width="0.3048" layer="1"/>
+<contactref element="IC1" pad="3"/>
+<via x="96.393" y="29.083" extent="1-16" drill="0.6"/>
+<wire x1="94.3578" y1="28.295" x2="95.605" y2="28.295" width="0.3048" layer="16"/>
+<wire x1="95.605" y1="28.295" x2="96.393" y2="29.083" width="0.3048" layer="16"/>
+<wire x1="97.9805" y1="30.6705" x2="96.393" y2="29.083" width="0.3048" layer="1"/>
 </signal>
 <signal name="5V">
@@
 <wire x1="89.5985" y1="8.001" x2="88.8365" y2="7.874" width="0.3048" layer="1"/>
 <wire x1="88.8365" y1="7.874" x2="83.2485" y2="13.462" width="0.3048" layer="1"/>
-<wire x1="83.2485" y1="13.462" x2="83.2485" y2="21.2725" width="0.3048" layer="1"/>
-<wire x1="83.2485" y1="21.2725" x2="82.55" y2="21.971" width="0.3048" layer="1"/>
 <via x="82.55" y="21.971" extent="1-16" drill="0.6"/>
 <wire x1="82.55" y1="21.971" x2="81.5975" y2="21.971" width="0.3048" layer="16"/>
@@
 <wire x1="81.3435" y1="21.717" x2="81.3435" y2="21.0955" width="0.3048" layer="16"/>
 <wire x1="81.3435" y1="21.0955" x2="81.3275" y2="21.0795" width="0.3048" layer="16"/>
+<wire x1="83.2485" y1="13.462" x2="83.2485" y2="16.383" width="0.3048" layer="1"/>
+<wire x1="83.2485" y1="16.383" x2="82.55" y2="17.0815" width="0.3048" layer="1"/>
+<wire x1="82.55" y1="21.971" x2="82.55" y2="17.0815" width="0.3048" layer="1"/>
 </signal>
 <signal name="GT3H">
@@
 <wire x1="96.3955" y1="33.1445" x2="96.393" y2="33.147" width="0.3048" layer="16"/>
 <wire x1="93.6625" y1="39.5605" x2="93.6625" y2="33.528" width="0.4064" layer="16"/>
-<wire x1="93.218" y1="27.6225" x2="93.218" y2="32.3215" width="0.4064" layer="16"/>
-<wire x1="93.218" y1="32.3215" x2="94.0435" y2="33.147" width="0.4064" layer="16"/>
 <wire x1="94.0435" y1="33.147" x2="96.393" y2="33.147" width="0.4064" layer="16"/>
 <wire x1="93.6625" y1="33.528" x2="94.0435" y2="33.147" width="0.4064" layer="16"/>
@@
 <wire x1="92.075" y1="27.559" x2="93.1545" y2="27.559" width="0.4064" layer="16"/>
 <wire x1="93.1545" y1="27.559" x2="93.218" y2="27.6225" width="0.4064" layer="16"/>
+<wire x1="93.218" y1="27.6225" x2="93.218" y2="29.972" width="0.4064" layer="16"/>
+<wire x1="93.218" y1="29.972" x2="96.393" y2="33.147" width="0.4064" layer="16"/>
 </signal>
 <signal name="N$34">
@@
 <via x="127.508" y="31.115" extent="1-16" drill="0.6"/>
 <wire x1="127.127" y1="31.496" x2="127.508" y2="31.115" width="0.3048" layer="1"/>
-<wire x1="88.5222" y1="27.645" x2="89.875" y2="27.645" width="0.3048" layer="16"/>
-<wire x1="89.875" y1="27.645" x2="89.9795" y2="27.7495" width="0.3048" layer="16"/>
 <wire x1="96.774" y1="22.4155" x2="95.377" y2="23.8125" width="0.3048" layer="1"/>
 <wire x1="95.377" y1="23.8125" x2="94.361" y2="23.8125" width="0.3048" layer="1"/>
 <wire x1="94.361" y1="23.8125" x2="92.2655" y2="25.8445" width="0.3048" layer="1"/>
-<wire x1="89.9795" y1="27.7495" x2="91.186" y2="27.7495" width="0.3048" layer="1"/>
-<wire x1="91.186" y1="27.7495" x2="92.2655" y2="26.67" width="0.3048" layer="1"/>
-<wire x1="92.2655" y1="25.8445" x2="92.2655" y2="26.67" width="0.3048" layer="1"/>
+<wire x1="89.9795" y1="27.7495" x2="92.0115" y2="27.7495" width="0.3048" layer="1"/>
+<wire x1="92.2655" y1="25.8445" x2="92.2655" y2="27.4955" width="0.3048" layer="1"/>
+<wire x1="92.2655" y1="27.4955" x2="92.0115" y2="27.7495" width="0.3048" layer="1"/>
+<wire x1="89.9795" y1="27.7495" x2="89.8525" y2="27.7495" width="0.3048" layer="16"/>
+<wire x1="89.8525" y1="27.7495" x2="89.789" y2="27.686" width="0.3048" layer="16"/>
+<wire x1="88.5222" y1="27.645" x2="89.875" y2="27.645" width="0.3048" layer="16"/>
+<wire x1="89.875" y1="27.645" x2="89.9795" y2="27.7495" width="0.3048" layer="16"/>
 </signal>
 </signals>
