File: hardware/cv-strip.sch (EAGLE design)
At the start: 83 parts, among them IC1 PIC16F1825SO14, IC2 74HC595D, IC3 MCP4728_QUAD_DAC, IC4 LM324D, IC5 REG1117, IC6 74HC595D

Commit message: getting there
Parts:
- removed JP1: (no value), pinhead:PINHD-1X2
- added U$2: PWR_SOCKET_2_1MM, jason_eagle6:PWR_SOCKET_2_1MM
Connections:
- net GND: now also U$2.PIN; no longer JP1.1
- net N$40: now also U$2.BARREL; no longer JP1.2
- net VOUTA: now also IC4B.+IN; no longer IC4C.+IN
- net VOUTB: now also IC4A.+IN; no longer IC4D.+IN
- net VOUTC: now also IC4D.+IN; no longer IC4A.+IN
- net VOUTD: now also IC4C.+IN; no longer IC4B.+IN
Changed lines of the file:
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@@
 <part name="GND23" library="supply1" deviceset="GND" device=""/>
 <part name="IC5" library="burr-brown" deviceset="REG1117" device=""/>
-<part name="JP1" library="pinhead" deviceset="PINHD-1X2" device=""/>
 <part name="GND4" library="supply1" deviceset="GND" device=""/>
 <part name="C11" library="resistor" deviceset="CPOL-EU" device="E2.5-5"/>
@@
 <part name="C6" library="rcl" deviceset="C-EU" device="C0805"/>
 <part name="GND8" library="supply1" deviceset="GND" device=""/>
+<part name="U$2" library="jason_eagle6" deviceset="PWR_SOCKET_2_1MM" device=""/>
 </parts>
 <sheets>
@@
 <instance part="GND23" gate="1" x="-15.24" y="-5.08"/>
 <instance part="IC5" gate="G$1" x="-58.42" y="208.28"/>
-<instance part="JP1" gate="G$1" x="-109.22" y="208.28" rot="R180"/>
 <instance part="GND4" gate="1" x="-58.42" y="187.96"/>
 <instance part="C11" gate="G$1" x="-81.28" y="200.66"/>
@@
 <instance part="C6" gate="G$1" x="76.2" y="116.84"/>
 <instance part="GND8" gate="1" x="76.2" y="106.68"/>
+<instance part="U$2" gate="G$1" x="-132.08" y="208.28"/>
 </instances>
 <busses>
@@
 </segment>
 <segment>
-<pinref part="JP1" gate="G$1" pin="1"/>
-<wire x1="-106.68" y1="205.74" x2="-83.82" y2="205.74" width="0.1524" layer="91"/>
+<wire x1="-114.3" y1="205.74" x2="-83.82" y2="205.74" width="0.1524" layer="91"/>
 <wire x1="-83.82" y1="205.74" x2="-83.82" y2="193.04" width="0.1524" layer="91"/>
 <pinref part="IC5" gate="G$1" pin="GND"/>
@@
 <junction x="-43.18" y="193.04"/>
 <pinref part="C5" gate="G$1" pin="-"/>
+<pinref part="U$2" gate="G$1" pin="PIN"/>
+<wire x1="-119.38" y1="213.36" x2="-114.3" y2="213.36" width="0.1524" layer="91"/>
+<wire x1="-114.3" y1="213.36" x2="-114.3" y2="205.74" width="0.1524" layer="91"/>
 </segment>
 <segment>
@@
 <net name="VOUTA" class="0">
 <segment>
-<label x="91.44" y="86.36" size="1.778" layer="95"/>
-<wire x1="106.68" y1="86.36" x2="93.98" y2="86.36" width="0.1524" layer="91"/>
-<pinref part="IC4" gate="C" pin="+IN"/>
-</segment>
-<segment>
 <pinref part="IC3" gate="G$1" pin="VOUTA"/>
 <wire x1="45.72" y1="71.12" x2="60.96" y2="71.12" width="0.1524" layer="91"/>
 <label x="58.42" y="71.12" size="1.778" layer="95"/>
 </segment>
+<segment>
+<pinref part="IC4" gate="B" pin="+IN"/>
+<wire x1="106.68" y1="101.6" x2="96.52" y2="101.6" width="0.1524" layer="91"/>
+<label x="96.52" y="101.6" size="1.778" layer="95"/>
+</segment>
 </net>
 <net name="VOUTB" class="0">
-<segment>
-<label x="93.98" y="71.12" size="1.778" layer="95"/>
-<wire x1="106.68" y1="71.12" x2="93.98" y2="71.12" width="0.1524" layer="91"/>
-<pinref part="IC4" gate="D" pin="+IN"/>
-</segment>
 <segment>
 <pinref part="IC3" gate="G$1" pin="VOUTB"/>
@@
 <label x="58.42" y="73.66" size="1.778" layer="95"/>
 </segment>
+<segment>
+<pinref part="IC4" gate="A" pin="+IN"/>
+<wire x1="106.68" y1="116.84" x2="96.52" y2="116.84" width="0.1524" layer="91"/>
+<label x="96.52" y="116.84" size="1.778" layer="95"/>
+</segment>
 </net>
 <net name="VOUTC" class="0">
-<segment>
-<label x="91.44" y="116.84" size="1.778" layer="95"/>
-<wire x1="106.68" y1="116.84" x2="93.98" y2="116.84" width="0.1524" layer="91"/>
-<pinref part="IC4" gate="A" pin="+IN"/>
-</segment>
 <segment>
 <pinref part="IC3" gate="G$1" pin="VOUTC"/>
@@
 <label x="58.42" y="76.2" size="1.778" layer="95"/>
 </segment>
+<segment>
+<pinref part="IC4" gate="D" pin="+IN"/>
+<wire x1="106.68" y1="71.12" x2="96.52" y2="71.12" width="0.1524" layer="91"/>
+<label x="96.52" y="71.12" size="1.778" layer="95"/>
+</segment>
 </net>
 <net name="VOUTD" class="0">
-<segment>
-<label x="93.98" y="101.6" size="1.778" layer="95"/>
-<wire x1="106.68" y1="101.6" x2="93.98" y2="101.6" width="0.1524" layer="91"/>
-<pinref part="IC4" gate="B" pin="+IN"/>
-</segment>
 <segment>
 <pinref part="IC3" gate="G$1" pin="VOUTD"/>
 <wire x1="45.72" y1="78.74" x2="60.96" y2="78.74" width="0.1524" layer="91"/>
 <label x="58.42" y="78.74" size="1.778" layer="95"/>
+</segment>
+<segment>
+<pinref part="IC4" gate="C" pin="+IN"/>
+<wire x1="106.68" y1="86.36" x2="96.52" y2="86.36" width="0.1524" layer="91"/>
+<label x="96.52" y="86.36" size="1.778" layer="95"/>
 </segment>
 </net>
@@
 <segment>
 <pinref part="D3" gate="1" pin="A"/>
-<pinref part="JP1" gate="G$1" pin="2"/>
-<wire x1="-91.44" y1="208.28" x2="-106.68" y2="208.28" width="0.1524" layer="91"/>
-</segment>
-</net>
+<wire x1="-91.44" y1="208.28" x2="-119.38" y2="208.28" width="0.1524" layer="91"/>
+<pinref part="U$2" gate="G$1" pin="BARREL"/>
+</segment>
+</net>

Commit message: almost done?
Parts:
- removed C22, C24: (no value), rcl:C-EUC0805
- removed R31, R32, R33: (no value), rcl:R-EU_R0805
- added C10, C13: (no value), rcl:C-EUC0805
- added R15, R16, R6: (no value), rcl:R-EU_R0805
- C11, C5: device resistor:CPOL-EUE2.5-5 -> rcl:C-EUC0805
- C20, C21: device rcl:C-EUC0805 -> resistor:CPOL-EUE2.5-5
- IC3: value MCP4728_QUAD_DAC -> 74HC595D; device jason_eagle6:MCP4728_QUAD_DAC -> 74xx-eu:74HC595D
- IC4: value LM324D -> MCP4728_QUAD_DAC; device linear:LM324D -> jason_eagle6:MCP4728_QUAD_DAC
- IC5: value REG1117 -> LM324D; device burr-brown:REG1117 -> linear:LM324D
- IC6: value 74HC595D -> REG1117; device 74xx-eu:74HC595D -> burr-brown:REG1117
- renumbered ACT to L1, C23 to C7, D3 to D2, DRMA to DRM1, GATA to CLK2, OK1 to IC7, PWR to L3, R30 to R11, R34 to R9, STS to L2, SYNC1 to CLK1, U$1 to D1
Connections:
- net GND: now also C10.1, C11.1, C12.2, C13.2, C17.2, C18.2, C19.1, C20.-, C21.-, C5.2, IC3A.G, IC3P.GND, IC4.LDAC#, IC4.VSS, IC5P.V-, IC6.GND, R1.2, R18.1, R19.1, R2.2, R24.1, R28.2, R3.2; no longer C11.-, C12.1, C17.1, C18.1, C19.2, C20.2, C21.2, C22.2, C24.2, C5.-, IC3.LDAC#, IC3.VSS, IC4P.V-, IC5.GND, IC6A.G, IC6P.GND, R10.2, R12.2, R13.2, R14.2, R20.1, R23.1, R28.1
- net MIDI_IN: now also R27.1; no longer R8.1
- net N$1: now also C16.1, R15.2; no longer C4.1, R4.2
- net N$12: now also IC3A.QA, R15.1; no longer IC2A.QA, R4.1
- net N$13: now also IC3A.QB, R16.1; no longer IC2A.QB, R3.1
- net N$15: now also IC3A.QD, R13.1; no longer IC2A.QD, R1.1
- net N$16: now also IC3A.QC, R14.1; no longer IC2A.QC, R2.1
- net N$2: now also IC5A.OUT, R17.2; no longer IC4A.OUT, R27.2
- net N$20: now also C4.1, R8.2; no longer C21.1, R32.2
- net N$21: now also IC4.SCL, R22.2; no longer IC3.SCL, R19.2
- net N$22: now also IC4.SDA, R21.2; no longer IC3.SDA, R18.2
- net N$23: now also C3.1, R7.2; no longer C15.1, R33.2
- net N$24: now also C2.1, R6.2; no longer C16.1, R17.2
- net N$25: now also IC5A.-IN, R17.1, R18.2; no longer IC4A.-IN, R27.1, R28.2
- net N$26: now also IC5B.-IN, R19.2, R20.1; no longer IC4B.-IN, R22.1, R23.2
- net N$27: now also IC5C.-IN, R25.2, R26.1; no longer IC4C.-IN, R20.2, R21.1
- net N$28: now also IC5D.-IN, R23.1, R24.2; no longer IC4D.-IN, R25.2, R26.1
- net N$29: now also R29.1; no longer R7.1
- net N$3: now also IC5B.OUT, R20.2; no longer IC4B.OUT, R22.2
- net N$30: now also R29.2; no longer R7.2
- net N$32: now also C1.1, R5.2; no longer C19.1, R24.2
- net N$33: now also C8.1, R12.2; no longer C20.1, R29.2
- net N$35: now also R1.1; no longer R14.1
- net N$36: now also R3.1; no longer R13.1
- net N$37: now also R2.1; no longer R12.1
- net N$4: now also IC5C.OUT, R26.2; no longer IC4C.OUT, R21.2
- net N$41: now also C6.1, R10.2; no longer C22.1, R31.2
- net N$42: now also R28.1; no longer R10.1
- net N$43: now also IC2A.QA, R8.1; no longer IC6A.QA, R32.1
- net N$46: now also IC2A.QB, R7.1; no longer IC6A.QB, R33.1
- net N$47: now also IC2A.QD, R5.1; no longer IC6A.QD, R24.1
- net N$48: now also IC2A.QC, R6.1; no longer IC6A.QC, R17.1
- net N$49: now also IC2A.QF; no longer IC6A.QF
- net N$5: now also IC5D.OUT, R23.2; no longer IC4D.OUT, R26.2
- net N$50: now also IC2A.QG, R10.1; no longer IC6A.QG, R31.1
- net N$51: now also IC2A.QE, R12.1; no longer IC6A.QE, R29.1
- net N$52: now also C5.1; no longer C24.1
- net N$53: now also IC2A.QH; no longer IC6A.QH
- net N$6: now also C17.1, R16.2; no longer C3.1, R3.2
- net N$7: now also C15.1, R14.2; no longer C2.1, R2.2
- net N$8: now also C14.1, R13.2; no longer C1.1, R1.2
- net N$9: now also R4.2; no longer R5.2
- net SR_CLK: now also IC3A.SCK; no longer IC6A.SCK
- net SR_DAT: now also IC3A.SER; no longer IC2A.SER
- net SR_DAT2: now also IC2A.SER; no longer IC6A.SER
- net SR_RCK: now also IC3A.RCK; no longer IC6A.RCK
- net VDD: now also C11.2, C12.1, C13.1, C19.2, C20.+, IC3A.SCL, IC3P.VCC, IC4.VDD, IC6.VOUT, R21.1, R22.1, R27.2, R4.1; no longer C12.2, C14.1, C17.2, C5.+, C8.1, IC3.VDD, IC5.VOUT, IC6A.SCL, IC6P.VCC, R18.1, R19.1, R5.1, R8.2
- net VIN: now also C10.2, C18.1, C21.+, IC5P.V+, IC6.VIN; no longer C11.+, C18.2, C6.1, IC4P.V+, IC5.VIN
- net VOUTA: now also IC4.VOUTA, IC5B.+IN; no longer IC3.VOUTA, IC4B.+IN
- net VOUTB: now also IC4.VOUTB, IC5A.+IN; no longer IC3.VOUTB, IC4A.+IN
- net VOUTC: now also IC4.VOUTC, IC5D.+IN; no longer IC3.VOUTC, IC4D.+IN
- net VOUTD: now also IC4.VOUTD, IC5C.+IN; no longer IC3.VOUTD, IC4C.+IN
Other:
- moved on the sheet: C1, C12, C14, C15, C16, C17, C18, C19, C2, C3, C4, C6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

Commit message: tweaks
Parts:
- renumbered ISCP to ICSP
Changed lines of the file:
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@@
 <part name="C16" library="rcl" deviceset="C-EU" device="C0805"/>
 <part name="GND16" library="supply1" deviceset="GND" device=""/>
-<part name="ISCP" library="tag-connect" deviceset="TC2030" device="-MCP-NL"/>
+<part name="ICSP" library="tag-connect" deviceset="TC2030" device="-MCP-NL"/>
 <part name="GND18" library="supply1" deviceset="GND" device=""/>
 <part name="GND19" library="supply1" deviceset="GND" device=""/>
@@
 <instance part="GND16" gate="1" x="114.3" y="-53.34"/>
 <instance part="IC5" gate="P" x="88.9" y="114.3"/>
-<instance part="ISCP" gate="G$1" x="-124.46" y="48.26" rot="MR0"/>
+<instance part="ICSP" gate="G$1" x="-124.46" y="48.26" rot="MR0"/>
 <instance part="GND18" gate="1" x="-93.98" y="33.02"/>
 <instance part="GND19" gate="1" x="7.62" y="58.42"/>
@@
 </segment>
 <segment>
-<pinref part="ISCP" gate="G$1" pin="VSS(GND)"/>
+<pinref part="ICSP" gate="G$1" pin="VSS(GND)"/>
 <wire x1="-111.76" y1="50.8" x2="-93.98" y2="50.8" width="0.1524" layer="91"/>
 <wire x1="-93.98" y1="50.8" x2="-93.98" y2="35.56" width="0.1524" layer="91"/>
@@
 <wire x1="-48.26" y1="86.36" x2="-45.72" y2="86.36" width="0.1524" layer="91"/>
 <junction x="-48.26" y="86.36"/>
-<pinref part="ISCP" gate="G$1" pin="ICSP_DAT/PGD"/>
+<pinref part="ICSP" gate="G$1" pin="ICSP_DAT/PGD"/>
 <wire x1="-111.76" y1="48.26" x2="-45.72" y2="48.26" width="0.1524" layer="91"/>
 <wire x1="-45.72" y1="86.36" x2="-33.02" y2="86.36" width="0.1524" layer="91"/>
@@
 <wire x1="-91.44" y1="81.28" x2="-93.98" y2="81.28" width="0.1524" layer="91"/>
 <wire x1="-93.98" y1="81.28" x2="-93.98" y2="55.88" width="0.1524" layer="91"/>
-<pinref part="ISCP" gate="G$1" pin="VPP/MCLR"/>
+<pinref part="ICSP" gate="G$1" pin="VPP/MCLR"/>
 <wire x1="-93.98" y1="55.88" x2="-111.76" y2="55.88" width="0.1524" layer="91"/>
 <junction x="-91.44" y="81.28"/>
@@
 <wire x1="-73.66" y1="96.52" x2="-99.06" y2="96.52" width="0.1524" layer="91"/>
 <junction x="-99.06" y="96.52"/>
-<pinref part="ISCP" gate="G$1" pin="VDD"/>
+<pinref part="ICSP" gate="G$1" pin="VDD"/>
 <wire x1="-111.76" y1="53.34" x2="-99.06" y2="53.34" width="0.1524" layer="91"/>
 <wire x1="-99.06" y1="53.34" x2="-99.06" y2="88.9" width="0.1524" layer="91"/>
@@
 <pinref part="IC1" gate="G$1" pin="RA1/ICPCLK"/>
 <junction x="-48.26" y="83.82"/>
-<pinref part="ISCP" gate="G$1" pin="ICSP_CLK/PGC"/>
+<pinref part="ICSP" gate="G$1" pin="ICSP_CLK/PGC"/>
 <wire x1="-111.76" y1="45.72" x2="-43.18" y2="45.72" width="0.1524" layer="91"/>
 <wire x1="-43.18" y1="83.82" x2="-33.02" y2="83.82" width="0.1524" layer="91"/>

Commit message: pcb v1
Other:
- note removed: "POLARITY TBC"
Changed lines of the file:
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@@
 <sheet>
 <plain>
-<text x="-96.52" y="320.04" size="5.08" layer="91">POLARITY TBC</text>
 </plain>
 <instances>
