File: hardware/cv-strip.sch (EAGLE design)
At the start: 118 parts, among them IC1 PIC16F1825SO14, IC2 AD5696R, IC3 MC14094B, IC4 MC14094B, IC5 LM324D, IC6 REG1117, IC7 6N138

Commit message: working on rev 3 LPC812
Parts:
- removed Q3, Q4, Q5, Q6: (no value), microbuilder:MOSFET-N_DUAL
- added C23: 100n, rcl:C-EUC0805
- added C24, C25: (no value), rcl:C-EUC0805
- added IC8: 24LC_64T-I/OT, Microchip-24LCxxx:24LC_64T-I/OT
- added IC9: MIC5504-2.8YM5-TR, jason_eagle6:MIC5504-2.8YM5-TR
- added Q15, Q16, Q17, Q18: (no value), jason_eagle6:MOSFET-N_DUAL
- IC1: value PIC16F1825SO14 -> LPC812; device jasons_stuff:PIC16F1825SO14 -> jason_eagle6:LPC812
Connections:
- net VIN renamed 12V
- removed net N$22: Q3G$1.G, R38.2
- removed net N$47: Q3G$2.G, R39.2
- removed net VDD: C10.1, C15.2, C16.+, C21.+, C9.2, D3.A, D4.A, IC1.VDD, IC2.GAIN, IC2.RESET#, IC2.VDD, IC2.VLOGIC, IC6.VOUT, IC7.VCC, ICSP.VDD, PWR.A, R21.1, R22.1, R27.2, R4.1
- new net 3V3: C15.1, C24.2, IC1.VDD, IC9.VOUT, ICSP.VDD, PWR.A, R4.1
- new net 5V: C10.1, C16.+, C21.+, C23.1, C25.2, C9.2, D3.A, D4.A, IC2.GAIN, IC2.RESET#, IC2.VDD, IC2.VLOGIC, IC6.VOUT, IC7.VCC, IC8.VCC, IC9.EN, IC9.VIN, R21.1, R22.1, R27.2, R38.2, R39.2
- new net MODE_SW: IC1.PIO0_17, MODE.S, MODE.S1
- new net N$57: IC1.PIO0_2/TMS, ICSP.ICSP_DAT/PGD
- new net N$58: IC1.RESET, ICSP.VPP/MCLR, R4.2
- net ACT_LED: now also IC1.PIO0_13; no longer IC1.RA2/INT
- net GND: now also C15.2, C23.2, C24.1, C25.1, IC8.VSS, IC8.WP, IC9.GND, Q15G$1.S, Q15G$2.S, Q16G$1.S, Q16G$2.S, Q17G$1.S, Q17G$2.S, Q18G$1.S, Q18G$2.S; no longer C15.1, Q3G$1.S, Q3G$2.S, Q4G$1.S, Q4G$2.S, Q5G$1.S, Q5G$2.S, Q6G$1.S, Q6G$2.S
- net GT1_VSEL: now also IC1.PIO0_16, Q18G$2.G; no longer IC1.RC4/TX
- net GT2_VSEL: now also IC1.PIO0_7, Q18G$1.G; no longer IC1.RC3/SS#
- net MIDI_IN: now also IC1.PIO0_4; no longer IC1.RC5/RX
- net N$14: now also Q15G$2.D; no longer Q6G$1.D
- net N$15: now also Q15G$1.D; no longer Q6G$2.D
- net N$16: now also Q16G$1.D; no longer Q5G$2.D
- net N$21: now also Q18G$1.D; no longer Q3G$2.D
- net N$34: now also IC1.PIO0_3/TCK, ICSP.ICSP_CLK/PGC; no longer IC1.RA3/MCLR#/VPP, ICSP.VPP/MCLR, MODE.S, MODE.S1, R4.2
- net N$48: now also Q16G$2.D; no longer Q5G$1.D
- net N$49: now also Q17G$2.D; no longer Q4G$1.D
- net N$50: now also Q17G$1.D; no longer Q4G$2.D
- net N$9: now also Q18G$2.D; no longer Q3G$1.D
- net SCL: now also IC1.PIO0_11, IC8.SCL; no longer IC1.RCO/SCL/SCK
- net SDA: now also IC1.PIO0_10, IC8.SDA; no longer IC1.RC1/SDA/SDI
- net SR_CLK: now also IC1.PIO0_15, Q16G$1.G, Q17G$1.G; no longer IC1.RA4/SDO, Q4G$2.G, Q5G$2.G
- net SR_DAT: now also IC1.PIO0_9, Q15G$1.G; no longer IC1.RA0/ICSPDAT, ICSP.ICSP_DAT/PGD, Q6G$2.G
- net SR_DAT2: now also IC1.PIO0_1, Q17G$2.G; no longer IC1.RA1/ICPCLK, ICSP.ICSP_CLK/PGC, Q4G$1.G
- net SR_RCK: now also IC1.PIO0_8, Q15G$2.G, Q16G$2.G; no longer IC1.RA5, Q5G$1.G, Q6G$1.G
- net STATUS_LED: now also IC1.PIO0_12; no longer IC1.RC2
Other:
- note added: "MIDI-TO-CV CONVERTER JASON HOTCHKISS SIXTY FOUR PIXELS LTD"
- note removed: "MIDI-TO-CV CONVERTER JASON HOTCHKISS SIXTY FOUR PIXELS LTD 13 JUN16"
- note removed: "PIC16F1825 MICRO CONTROLLER"
- moved on the sheet: C15, MODE, R21, R22, R38, R39, R4

Commit message: mods
Parts:
- renumbered Q15 to Q6, Q16 to Q5, Q17 to Q4, Q18 to Q3
Connections:
- net MIDI_IN: now also IC1.PIO0_0; no longer IC1.PIO0_4
- net STATUS_LED: now also IC1.PIO0_14; no longer IC1.PIO0_12

Commit message: rev3 PCB final
Connections:
- net SCL: now also IC1.PIO0_10; no longer IC1.PIO0_11
- net SDA: now also IC1.PIO0_11; no longer IC1.PIO0_10
- net STATUS_LED: now also IC1.PIO0_12; no longer IC1.PIO0_14
Changed lines of the file:
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@@
 <segment>
 <pinref part="R22" gate="G$1" pin="2"/>
-<wire x1="-99.06" y1="60.96" x2="-129.54" y2="60.96" width="0.1524" layer="91"/>
-<wire x1="-129.54" y1="60.96" x2="-132.08" y2="60.96" width="0.1524" layer="91"/>
-<wire x1="-129.54" y1="88.9" x2="-129.54" y2="60.96" width="0.1524" layer="91"/>
-<junction x="-129.54" y="60.96"/>
-<label x="-134.62" y="60.96" size="1.778" layer="95"/>
-<pinref part="IC1" gate="G$1" pin="PIO0_11"/>
-<junction x="-99.06" y="60.96"/>
+<wire x1="-129.54" y1="58.42" x2="-132.08" y2="58.42" width="0.1524" layer="91"/>
+<wire x1="-129.54" y1="88.9" x2="-129.54" y2="58.42" width="0.1524" layer="91"/>
+<junction x="-129.54" y="58.42"/>
+<label x="-134.62" y="58.42" size="1.778" layer="95"/>
+<pinref part="IC1" gate="G$1" pin="PIO0_10"/>
+<wire x1="-129.54" y1="58.42" x2="-99.06" y2="58.42" width="0.1524" layer="91"/>
+<junction x="-99.06" y="58.42"/>
 </segment>
 <segment>
@@
 <segment>
 <pinref part="R21" gate="G$1" pin="2"/>
-<wire x1="-132.08" y1="58.42" x2="-127" y2="58.42" width="0.1524" layer="91"/>
-<wire x1="-127" y1="88.9" x2="-127" y2="58.42" width="0.1524" layer="91"/>
-<junction x="-127" y="58.42"/>
-<label x="-134.62" y="58.42" size="1.778" layer="95"/>
-<pinref part="IC1" gate="G$1" pin="PIO0_10"/>
-<wire x1="-127" y1="58.42" x2="-99.06" y2="58.42" width="0.1524" layer="91"/>
-<junction x="-99.06" y="58.42"/>
+<wire x1="-132.08" y1="60.96" x2="-127" y2="60.96" width="0.1524" layer="91"/>
+<wire x1="-127" y1="88.9" x2="-127" y2="60.96" width="0.1524" layer="91"/>
+<junction x="-127" y="60.96"/>
+<label x="-134.62" y="60.96" size="1.778" layer="95"/>
+<pinref part="IC1" gate="G$1" pin="PIO0_11"/>
+<wire x1="-127" y1="60.96" x2="-99.06" y2="60.96" width="0.1524" layer="91"/>
+<junction x="-99.06" y="60.96"/>
 </segment>
 <segment>
@@
 </segment>
 <segment>
-<label x="-58.42" y="78.486" size="1.778" layer="95"/>
-<pinref part="IC1" gate="G$1" pin="PIO0_14"/>
-<wire x1="-63.5" y1="78.74" x2="-58.42" y2="78.74" width="0.1524" layer="91"/>
-<junction x="-63.5" y="78.74"/>
+<label x="-116.332" y="73.66" size="1.778" layer="95"/>
+<pinref part="IC1" gate="G$1" pin="PIO0_12"/>
+<wire x1="-104.14" y1="73.66" x2="-99.06" y2="73.66" width="0.1524" layer="91"/>
+<junction x="-99.06" y="73.66"/>
 </segment>
 </net>
@@
 <label x="-58.42" y="70.866" size="1.778" layer="95"/>
 <pinref part="IC1" gate="G$1" pin="PIO0_7"/>
-<wire x1="-63.5" y1="71.12" x2="-58.42" y2="71.12" width="0.1524" layer="91"/>
+<wire x1="-63.5" y1="71.12" x2="-60.96" y2="71.12" width="0.1524" layer="91"/>
 <junction x="-63.5" y="71.12"/>
-</segment>
-</net>
+<junction x="-60.96" y="71.12"/>
+<wire x1="-60.96" y1="71.12" x2="-58.42" y2="71.12" width="0.1524" layer="91"/>
+</segment>
+</net>

Commit message: label changes only
Other:
- note added: "0V/5V or 0V/12V outputs depending on supply voltage to shift register"
- note added: "24LC64T-I/OT 64KBIT"
- note added: "3.5mm MIDI jack with +5V tip (e.g. Novation/Arturia) can be used as alternative to MIDI DIN input (not both at same time)"
- note added: "AD5696RARUZ 16-Bit DAC"
- note added: "CV OUTPUT DAC"
- note added: "CV-OCD rev 3 MIDI-TO-CV CONVERTER JASON HOTCHKISS SIXTY FOUR PIXELS LTD"
- note added: "D3/D4 Schottky Rectifier"
- note added: "D5 Schottky Rectifier"
- note added: "LPC812 MCU (CORTEX M0+)"
- note added: "Logic low input enables 12V supply to gate shift registers."
- note added: "MC14094BDR2G CMOS Shift Register"
- note added: "POWER SUPPLY"
- note added: "SERIAL EEPROM"
- note added: "TLV2374QDRG4Q1 Op-Amp R2R"
- note added: "Tristate outputs 0V/Hi-Z/5V or 0V/Hi-Z/12V depending on supply voltage to shift register IC"
- note removed: "CV OUTPUT 16-BIT DAC"
- note removed: "MIDI-TO-CV CONVERTER JASON HOTCHKISS SIXTY FOUR PIXELS LTD"
- note removed: "POWER SUPPLY REGULATOR"
- moved on the sheet: ACT, C24, C25, PWR, R1, R2, R3, STA
