File: cvocd_banana/cvocd_banana.kicad_pcb (KiCad board)
At the start: 2 copper layers, 230 x 95 mm, 158 parts, among them SW1 SW_SP3T, SW2 SW_SP3T, SW3 SW_SP3T, U1 4504, U2 4504, U3 4504, U4 LM324, U5 MC34063AD, U6 LM317L_SOT-89, U7 AMS1117

Commit message: ASD
Parts:
- renumbered U1 to IC1, U2 to IC2, U3 to IC3, U4 to IC4, U5 to IC5, U6 to IC6, U7 to IC7, R13 to R11, R11 to R12, R12 to R13, R20 to R19, R3 to R2, R19 to R20, R23 to R22, R22 to R23, R5 to R3, R6 to R5, R7 to R6, R2 to R7, XG2 to XG1, XG9 to XG10, XG10 to XG11, XG11 to XG12, XG3 to XG2, XG4 to XG3, XG1 to XG4, XG8 to XG5, XG5 to XG6, XG6 to XG7, XG7 to XG8, XG12 to XG9
Connections:
- IC1 pad 11: unconnected-(U1-Ein-Pad11) -> GND
- IC1 pad 9: unconnected-(U1-Din-Pad9) -> GND
Other:
- board text added: "CVA"
- board text added: "CVB"
- board text added: "CVC"
- board text added: "CVD"
- board text added: "GND"
- board text added: "MIDI LED"
- board text added: "MODE SWITCH"
- board text added: "STATUS LED"
- board text added: "VIN"

Commit message: REV1
Parts:
- added GND4: Conn_01x01, Jason_Kicad:WireToBoardCVOCD, F.Cu at (52.8, 140.8)
- added POWER3: Conn_01x01, Jason_Kicad:WireToBoardCVOCD, F.Cu at (99.8, 141.0)
- added POWER4: Conn_01x01, Jason_Kicad:WireToBoardCVOCD, F.Cu at (76.5, 141.0)
- added POWER5: Conn_01x01, Jason_Kicad:WireToBoardCVOCD, F.Cu at (59.2, 140.8)
- renumbered XG11 to GATE10X1, XG12 to GATE11X1, XG9 to GATE12X1, XG4 to GATE1X1, XG1 to GATE2X1, XG2 to GATE3X1, XG3 to GATE4X1, XG6 to GATE5X1, XG7 to GATE6X1, XG8 to GATE7X1, XG5 to GATE8X1, XG10 to GATE9X1
Routing:
- net +10V: track 69.3 -> 84.0 mm
- net +15V: track 121.7 -> 130.8 mm
- net +5V: track 448.5 -> 455.9 mm
- net GND: track 5.47 -> 8.46 mm
Other:
- board text added: "10"
- board text added: "10V"
- board text added: "15"
- board text added: "15V"
- board text added: "5"
- board text added: "5V"
- board text added: "ACT"
- board text added: "BTN"
- board text added: "CVOCD BANANA BREAKOUT/GATE BOOST REV 1"
- board text added: "GT1"
- board text added: "GT1 -4"
- board text added: "GT10"
- board text added: "GT11"
- board text added: "GT12"
- board text added: "GT2"
- board text added: "GT3"
- board text added: "GT4"
- board text added: "GT5"
- board text added: "GT5 -8"
- board text added: "GT6"
- board text added: "GT7"
- board text added: "GT8"
- board text added: "GT9"
- board text added: "GT9 -12"
- board text added: "MIDI"
- board text added: "MIDI IN"
- board text added: "P4"
- board text added: "P5"
- board text added: "PWR"
- board text added: "SIX4PIX.COM"
- board text added: "SNK"
- board text added: "SRC"
- board text added: "STAT"
- board text added: "SW"
- board text removed: "MIDI LED"
- board text removed: "MODE SWITCH"
- board text removed: "STATUS LED"

Commit message: updates to banana pcb
Parts:
- added D1: D_Zener, Diode_SMD:D_0805_2012Metric, F.Cu at (221.0, 125.8)
- added D2: D_Zener, Diode_SMD:D_0805_2012Metric, F.Cu at (208.5, 125.8)
- added D3: D_Zener, Diode_SMD:D_0805_2012Metric, F.Cu at (221.0, 113.0)
- added D4: D_Zener, Diode_SMD:D_0805_2012Metric, F.Cu at (208.5, 113.0)
- added Q1: 2N7002, Package_TO_SOT_SMD:SOT-23, F.Cu at (221.0, 129.2)
- added Q2: 2N7002, Package_TO_SOT_SMD:SOT-23, F.Cu at (208.5, 129.2)
- added Q3: 2N7002, Package_TO_SOT_SMD:SOT-23, F.Cu at (221.0, 116.5)
- added Q4: 2N7002, Package_TO_SOT_SMD:SOT-23, F.Cu at (208.5, 116.5)
- added R42: R, Resistor_SMD:R_0805_2012Metric, F.Cu at (101.5, 118.0)
- added SW4: SW_SPDT, Jason_Kicad:Slide_1P2T_Rev_Mnt_CLSB12B01, F.Cu at (105.0, 121.2)
- SW1, SW2, SW3: footprint Jason_Kicad:Slide_SW_Rev_Mnt_CLSB13B01 -> Jason_Kicad:Slide_1P3T_Rev_Mnt_CLSB13B01
- moved XMIDI1 4.61 mm to (246.5, 74.5)
- moved XMIDI2 4.61 mm to (242.0, 74.5)
- renumbered D1 to D5, D2 to D6, D3 to D7, D4 to D8, D5 to D9
Connections:
- SW1 pad 1: +15V -> unconnected-(SW1-Pad1)
- SW1 pad 4: unconnected-(SW1-Pad4) -> +15V
- SW2 pad 1: +15V -> unconnected-(SW2-Pad1)
- SW2 pad 4: unconnected-(SW2-Pad4) -> +15V
- SW3 pad 1: +15V -> unconnected-(SW3-Pad1)
- SW3 pad 4: unconnected-(SW3-Pad4) -> +15V
Routing:
- net CLAMP_EN: track 0.00 -> 157.5 mm, vias 0 -> 2
- net +5V: track 455.9 -> 474.8 mm, vias 10 -> 11
- net +15V: track 130.8 -> 114.6 mm
- net Net-(MIDI1-Pin_1): track 83.0 -> 76.9 mm
- net Net-(MIDI2-Pin_1): track 78.7 -> 84.7 mm
- net CV1: track 47.1 -> 51.4 mm
- net CV3: track 72.5 -> 76.8 mm
- net CV2: track 77.6 -> 81.9 mm
- net CV4: track 103.0 -> 107.2 mm
- net Net-(D1-A): track 0.00 -> 3.00 mm
- net Net-(D4-A): track 0.00 -> 2.95 mm
- net Net-(D3-A): track 0.00 -> 2.95 mm
- net Net-(D2-A): track 0.00 -> 2.95 mm
- net VIN: track 146.8 -> 144.2 mm
- net GATE7: track 134.5 -> 136.1 mm
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Other:
- board text added: "CV LMT"
- board text added: "N"
- board text added: "P4+"
- board text added: "P5-"
- board text added: "Y"
- board text removed: "P4"
- board text removed: "P5"

Commit message: fascia
Parts:
- added REF**: MountingHole_3.2mm_M3, MountingHole:MountingHole_3.2mm_M3, F.Cu at (145.0, 53.2)
- moved C10 11.5 mm to (143.0, 66.5)
- moved R12 8.94 mm to (135.0, 53.5)
Routing:
- net Net-(IC2-Dout): track 91.0 -> 79.6 mm
- net Net-(GATE5X1-Pin_1): track 7.79 -> 17.6 mm
- net GND: vias 25 -> 28
Changed lines of the file:
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@@
 	(footprint "Resistor_SMD:R_0805_2012Metric"
 		(layer "F.Cu")
-		(at 143 57.5)
+		(at 135 53.5)
 		(descr "Resistor SMD 0805 (2012 Metric), square (rectangular) end terminal, IPC_7351 nominal, (Body size source: IPC-SM-782 page 72, https://www.pcb-3d.com/wordpress/wp-content/uploads/ipc-sm-782a_amendment_1_and_2.pdf), generated with kicad-footprint-generator")
 		(tags "resistor")
@@
 		(tags "diode")
 		(property "Reference" "D1"
-			(at -3 0 360)
+			(at -3 0 0)
 			(layer "F.SilkS")
 			(effects
@@
 		)
 		(property "Value" "D_Zener"
-			(at 0 1.65 360)
+			(at 0 1.65 0)
 			(layer "F.Fab")
 			(effects
@@
 		)
 		(fp_text user "${REFERENCE}"
-			(at 0 0 360)
+			(at 0 0 0)
 			(layer "F.Fab")
 			(effects
@@
 	(footprint "Capacitor_SMD:C_0805_2012Metric"
 		(layer "F.Cu")
-		(at 143 55)
+		(at 143 66.5)
 		(descr "Capacitor SMD 0805 (2012 Metric), square (rectangular) end terminal, IPC_7351 nominal, (Body size source: IPC-SM-782 page 76, https://www.pcb-3d.com/wordpress/wp-content/uploads/ipc-sm-782a_amendment_1_and_2.pdf, https://docs.google.com/spreadsheets/d/1BsfQQcO9C6DZCsRaXUlFlo91Tg2WpOkGARC1WS5S8t0/edit?usp=sharing), generated with kicad-footprint-generator")
 		(tags "capacitor")
@@
 		)
 	)
+	(footprint "MountingHole:MountingHole_3.2mm_M3"
+		(layer "F.Cu")
+		(at 145 53.25)
+		(descr "Mounting Hole 3.2mm, no annular, M3")
+		(tags "mounting hole 3.2mm no annular m3")
+		(property "Reference" "REF**"
+			(at 0 -4.2 0)
+			(layer "F.SilkS")
+			(hide yes)
+			(effects
+				(font
+					(size 1 1)
+					(thickness 0.15)
+				)
+			)
+		)
+		(property "Value" "MountingHole_3.2mm_M3"
+			(at 0 4.2 0)
+			(layer "F.Fab")
+			(effects
+				(font
+					(size 1 1)
+					(thickness 0.15)
+				)
+			)
+		)
+		(property "Footprint" "MountingHole:MountingHole_3.2mm_M3"
+			(at 0 0 0)
+			(unlocked yes)
+			(layer "F.Fab")
+			(hide yes)
+			(effects
+				(font
+					(size 1.27 1.27)
+					(thickness 0.15)
+				)
+			)
+		)
+		(property "Datasheet" ""
+			(at 0 0 0)
+			(unlocked yes)
+			(layer "F.Fab")
+			(hide yes)
+			(effects
+				(font
+					(size 1.27 1.27)
+					(thickness 0.15)
+				)
+			)
+		)
+		(property "Description" ""
+			(at 0 0 0)
+			(unlocked yes)
+			(layer "F.Fab")
+			(hide yes)
+			(effects
+				(font
+					(size 1.27 1.27)
+					(thickness 0.15)
+				)
+			)
+		)
+		(attr board_only)
+		(fp_circle
+			(center 0 0)
+			(end 3.2 0)
+			(stroke
+				(width 0.15)
+				(type solid)
+			)
+			(fill none)
+			(layer "Cmts.User")
+		)
+		(fp_circle
+			(center 0 0)
+			(end 3.45 0)
+			(stroke
+				(width 0.05)
+				(type solid)
+			)
+			(fill none)
+			(layer "F.CrtYd")
+		)
+		(fp_text user "${REFERENCE}"
+			(at 0 0 0)
+			(layer "F.Fab")
+			(effects
+				(font
+					(size 1 1)
+					(thickness 0.15)
+				)
+			)
+		)
+		(pad "" np_thru_hole circle
+			(at 0 0)
+			(size 3.2 3.2)
+			(drill 3.2)
+			(layers "*.Cu" "*.Mask")
+		)
+	)
 	(footprint "Resistor_SMD:R_0805_2012Metric"
 		(layer "F.Cu")
@@
 	)
 	(via
+		(at 186.5 84.25)
+		(size 0.9)
+		(drill 0.6)
+		(layers "F.Cu" "B.Cu")
+		(free yes)
+		(net 2)
+	)
+	(via
 		(at 63.5 112)
 		(size 0.9)
@@
 	)
 	(via
+		(at 209.5 84.25)
+		(size 0.9)
+		(drill 0.6)
+		(layers "F.Cu" "B.Cu")
+		(free yes)
+		(net 2)
+	)
+	(via
 		(at 91.8 138.2)
 		(size 0.9)
@@
 	)
 	(via
+		(at 167.5 83.75)
+		(size 0.9)
+		(drill 0.6)
+		(layers "F.Cu" "B.Cu")
+		(free yes)
+		(net 2)
+	)
+	(via
 		(at 54.0875 108.5)
 		(size 0.9)
@@
 	)
 	(segment
-		(start 140.5 57.5)
-		(end 142.0875 57.5)
-		(width 0.3)
-		(layer "F.Cu")
-		(net 63)
-	)
-	(segment
 		(start 67.825 63.675)
 		(end 68.5 63)
@@
 	)
 	(segment
-		(start 68.5 63)
-		(end 68.5 54)
-		(width 0.3)
-		(layer "F.Cu")
-		(net 63)
-	)
-	(segment
-		(start 139.5 53.5)
-		(end 140 54)
-		(width 0.3)
-		(layer "F.Cu")
-		(net 63)
-	)
-	(segment
 		(start 69 53.5)
-		(end 139.5 53.5)
-		(width 0.3)
-		(layer "F.Cu")
-		(net 63)
-	)
-	(segment
-		(start 140 57)
-		(end 140.5 57.5)
+		(end 134.0875 53.5)
 		(width 0.3)
 		(layer "F.Cu")
@@
 	)
 	(segment
-		(start 140 54)
-		(end 140 57)
+		(start 63.975 63.675)
+		(end 67.825 63.675)
 		(width 0.3)
 		(layer "F.Cu")
@@
 	)
 	(segment
-		(start 63.975 63.675)
-		(end 67.825 63.675)
+		(start 68.5 63)
+		(end 68.5 54)
 		(width 0.3)
 		(layer "F.Cu")
@@
 	)
 	(segment
-		(start 143.25 62.5)
-		(end 143.25 59.75)
+		(start 143.95 65.45)
+		(end 143.25 64.75)
 		(width 0.3)
 		(layer "F.Cu")
@@
 	)
 	(segment
-		(start 143.9125 57.5)
-		(end 143.9125 55.0375)
+		(start 138 53.5)
+		(end 135.9125 53.5)
+		(width 0.3)
+		(layer "F.Cu")
+		(net 88)
+	)
+	(segment
+		(start 143.25 62.5)
+		(end 143.25 58.75)
 		(width 0.3)
 		(layer "F.Cu")
@@
 	)
 	(segment
-		(start 143.25 59.75)
-		(end 143.9125 59.0875)
+		(start 143.25 64.75)
+		(end 143.25 62.5)
 		(width 0.3)
 		(layer "F.Cu")
@@
 	)
 	(segment
-		(start 143.9125 59.0875)
-		(end 143.9125 57.5)
+		(start 143.95 66.5)
+		(end 143.95 65.45)
 		(width 0.3)
 		(layer "F.Cu")
@@
 	)
 	(segment
-		(start 143.9125 55.0375)
-		(end 143.95 55)
+		(start 143.25 58.75)
+		(end 138 53.5)
 		(width 0.3)
 		(layer "F.Cu")
