File: cvocd_banana/cvocd_banana.kicad_pcb (KiCad board)
At the start: 2 copper layers, 230 x 95 mm, 173 parts, among them IC1 4504, IC2 4504, IC3 4504, IC4 LM324, IC5 MC34063AD, IC6 LM317L_SOT-89, IC7 AMS1117, Q1 2N7002, Q2 2N7002, Q3 2N7002, Q4 2N7002, SW1 SW_SP3T, SW2 SW_SP3T, SW3 SW_SP3T, SW4 SW_SPDT

Commit message: pcb and fascia version 1
Routing:
- net GND: vias 28 -> 35
Changed lines of the file:
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@@
 			(outputformat 1)
 			(mirror no)
-			(drillshape 1)
+			(drillshape 0)
 			(scaleselection 1)
-			(outputdirectory "")
+			(outputdirectory "gerber")
 		)
 	)
@@
 	)
 	(via
+		(at 88.5 116.5)
+		(size 0.9)
+		(drill 0.6)
+		(layers "F.Cu" "B.Cu")
+		(free yes)
+		(net 2)
+	)
+	(via
 		(at 59.525 91.175)
 		(size 0.9)
@@
 	)
 	(via
+		(at 78.5 116.5)
+		(size 0.9)
+		(drill 0.6)
+		(layers "F.Cu" "B.Cu")
+		(free yes)
+		(net 2)
+	)
+	(via
+		(at 79.5 123.25)
+		(size 0.9)
+		(drill 0.6)
+		(layers "F.Cu" "B.Cu")
+		(free yes)
+		(net 2)
+	)
+	(via
 		(at 241.75 81.5)
 		(size 0.9)
@@
 	)
 	(via
+		(at 98.25 116.5)
+		(size 0.9)
+		(drill 0.6)
+		(layers "F.Cu" "B.Cu")
+		(free yes)
+		(net 2)
+	)
+	(via
 		(at 63.5 112)
 		(size 0.9)
@@
 	)
 	(via
+		(at 98 123.25)
+		(size 0.9)
+		(drill 0.6)
+		(layers "F.Cu" "B.Cu")
+		(free yes)
+		(net 2)
+	)
+	(via
 		(at 58.7 137.7)
 		(size 0.9)
@@
 		(size 0.9)
 		(drill 0.6)
+		(layers "F.Cu" "B.Cu")
+		(free yes)
+		(net 2)
+	)
+	(via
+		(at 89.75 123.25)
+		(size 0.9)
+		(drill 0.6)
+		(layers "F.Cu" "B.Cu")
+		(free yes)
+		(net 2)
+	)
+	(via
+		(at 75 82.25)
+		(size 0.9)
+		(drill 0.6)

Commit message: banana updates
Parts:
- removed the C21 at (47.0, 105.5)
- removed the C22 at (39.0, 112.0)
- removed the IC5 at (52.5, 104.0)
- removed the R38 at (55.0, 108.5)
- removed the R39 at (55.0, 111.0)
- added C24: C, Capacitor_SMD:C_1210_3225Metric_Pad1.33x2.70mm_HandSolder, F.Cu at (50.5, 103.0)
- added C25: C, Capacitor_SMD:C_1210_3225Metric_Pad1.33x2.70mm_HandSolder, F.Cu at (35.2, 103.0)
- added IC6: AP3012, Package_TO_SOT_SMD:SOT-23-5, F.Cu at (45.5, 108.5)
- added REF**: MountingHole_3.2mm_M3, MountingHole:MountingHole_3.2mm_M3, F.Cu at (145.0, 141.8)
- C22: renamed from C29; footprint Capacitor_SMD:CP_Elec_6.3x5.8 -> Capacitor_Tantalum_SMD:CP_EIA-6032-28_Kemet-C
- C23: footprint Capacitor_SMD:CP_Elec_6.3x5.8 -> Capacitor_Tantalum_SMD:CP_EIA-6032-28_Kemet-C
- C26: renamed from C20; footprint Capacitor_SMD:CP_Elec_6.3x5.8 -> Capacitor_Tantalum_SMD:CP_EIA-6032-28_Kemet-C
- C29: renamed from C26; footprint Capacitor_SMD:CP_Elec_6.3x5.8 -> Capacitor_Tantalum_SMD:CP_EIA-6032-28_Kemet-C
- L1: footprint Inductor_SMD:L_10.4x10.4_H4.8 -> Inductor_SMD:L_Taiyo-Yuden_MD-4040
- R36: value R -> 22k
- R37: value R -> 2k
- R38: renamed from R40; value R -> 470
- R39: renamed from R41; value R -> 3K3
- moved R36 19.5 mm to (39.0, 108.5), turned to -90 degrees
- moved R37 15.4 mm to (41.5, 108.5), turned to 90 degrees
- moved C20 15.2 mm to (67.8, 141.5), turned to 0 degrees
- moved C28 15.0 mm to (83.0, 141.5), turned to 180 degrees
- moved D6 14.0 mm to (39.0, 103.0), turned to 90 degrees
- moved C26 8.49 mm to (56.0, 103.5), turned to 90 degrees
- moved L1 6.08 mm to (45.5, 103.0), turned to 180 degrees
- moved XSW1 4.00 mm to (151.0, 141.5)
- moved XMIDILED1 3.00 mm to (138.0, 141.5)
- moved XSTATUSLED1 3.00 mm to (132.0, 141.5)
- moved XMIDI1 1.50 mm to (246.5, 76.0)
- moved XMIDI2 1.50 mm to (242.0, 76.0)
- renumbered C27 to C20, C28 to C21, C24 to C27, C25 to C28, IC7 to IC5, IC6 to IC7, R42 to R40
Connections:
- C19 pad 1: +5V -> +10V
- C20 pad 1: +10V -> Net-(D5-K)
- IC4 pad 4: +5V -> +10V
- IC5 pad 3: +10V -> Net-(D5-K)
- L1 pad 1: Net-(IC5-Ipk) -> Net-(D5-K)
- R36 pad 1: Net-(D5-K) -> Net-(D6-K)
- R36 pad 2: Net-(IC5-Ipk) -> Net-(IC6-FB)
- R37 pad 1: Net-(IC5-DC) -> Net-(IC6-FB)
- R37 pad 2: Net-(IC5-Ipk) -> GND
- SW4 pad 1: GND -> unconnected-(SW4-A-Pad1)
- SW4 pad 3: unconnected-(SW4-C-Pad3) -> GND
Routing:
- net +10V: track 84.0 -> 255.9 mm, vias 0 -> 2
- net Net-(D5-K): track 47.0 -> 97.9 mm, vias 0 -> 2
- net Net-(IC5-Ipk): track 27.8 -> 0.00 mm
- net +5V: track 474.8 -> 448.1 mm
- net Net-(D6-K): track 20.7 -> 35.4 mm
- net Net-(D6-A): track 17.5 -> 10.3 mm
- net Net-(IC5-Vfb): track 6.10 -> 0.00 mm
- net Net-(IC6-FB): track 0.00 -> 5.38 mm
- net Net-(IC5-TC): track 3.51 -> 0.00 mm
- net Net-(IC5-DC): track 3.50 -> 0.00 mm
- net Net-(MIDI2-Pin_1): track 84.7 -> 81.2 mm
- net GATE11: track 122.9 -> 125.7 mm
- net Net-(XMIDILED1-Pin_1): track 178.8 -> 181.5 mm
- net Net-(XSTATUSLED1-Pin_1): track 173.8 -> 176.5 mm
- net GATE10: track 121.7 -> 124.4 mm
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Other:
- board text added: "CVOCD BANANA BREAKOUT/GATE BOOST REV 2"
- board text removed: "CVOCD BANANA BREAKOUT/GATE BOOST REV 1"
- board text removed: "MIDI"

Commit message: banana pcb main v2
Parts:
- added REF**: Stencil8_mounting_hole, Jason_Kicad:Stencil8_mounting_hole, F.Cu at (35.0, 42.0)
- added REF**: Stencil8_mounting_hole, Jason_Kicad:Stencil8_mounting_hole, F.Cu at (255.0, 152.0)
- added REF**: Stencil8_mounting_hole, Jason_Kicad:Stencil8_mounting_hole, F.Cu at (255.0, 42.0)
- added REF**: Stencil8_mounting_hole, Jason_Kicad:Stencil8_mounting_hole, F.Cu at (35.0, 152.0)
- C10, C11, C12, C15, C16, C17, C18, C3, C4, C5, C6, C9: value C -> 10n
- C20, C21, C27, C28: value C -> 100n
- C22: value C_Polarized -> 100u; footprint Capacitor_Tantalum_SMD:CP_EIA-6032-28_Kemet-C -> Capacitor_Tantalum_SMD:CP_EIA-7343-31_Kemet-D
- C23, C26, C29: value C_Polarized -> 100u/20; footprint Capacitor_Tantalum_SMD:CP_EIA-6032-28_Kemet-C -> Capacitor_Tantalum_SMD:CP_EIA-7343-31_Kemet-D
- C24, C25: value C -> 1u; footprint Capacitor_SMD:C_1210_3225Metric_Pad1.33x2.70mm_HandSolder -> Capacitor_SMD:C_0805_2012Metric
- D1, D2, D3, D4: value D_Zener -> 5V1
- D7, D8, D9: value D_Schottky -> MBR0520
- L1: value L -> TYS4012100M-10/10uH
- L2: value L -> CM322522-1R0KL/1uH
- R33, R34, R35: value R -> 1k
- R40: value R -> 10k
- moved C25 2.25 mm to (37.5, 103.0)
- moved D6 1.50 mm to (40.5, 103.0)
Routing:
- net Net-(D6-K): track 35.4 -> 39.6 mm
- net Net-(D6-A): track 10.3 -> 8.99 mm
- net Net-(D5-K): track 97.9 -> 98.4 mm
Other:
- board size 230 x 95 mm -> 230 x 116 mm
- board text added: "1"
- board text added: "11"
- board text added: "12"
- board text added: "2"
- board text added: "3"
- board text added: "4"
- board text added: "6"
- board text added: "7"
- board text added: "8"
- board text added: "9"
- board text added: "A"
- board text added: "B"
- board text added: "C"
- board text added: "D"
- board text added: "MIDI"
- board text added: "STA"
- board text removed: "CVA"
- board text removed: "CVB"
- board text removed: "CVC"
- board text removed: "CVD"
- board text removed: "GT1"
- board text removed: "GT10"
- board text removed: "GT11"
- board text removed: "GT12"
- board text removed: "GT2"
- board text removed: "GT3"
- board text removed: "GT4"
- board text removed: "GT5"
- board text removed: "GT6"
- board text removed: "GT7"
- board text removed: "GT8"
- board text removed: "GT9"
