File: cvocd_banana/cv_out.kicad_sch (KiCad schematic)
At the start: 18 parts, among them U4 LM324

Commit message: ASD
Parts:
- renumbered U4 to IC4
Changed lines of the file:
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@@
 		(dnp no)
 		(fields_autoplaced yes)
-		(property "Reference" "U4"
+		(property "Reference" "IC4"
 			(at 73.66 49.5299 0)
 			(effects
@@
 			(project ""
 				(path "/d6028aad-759f-4736-9818-30f0061d1d8d/721fd379-0889-4e74-8212-a23ae46bf4ef"
-					(reference "U4")
+					(reference "IC4")
 					(unit 5)
 				)
@@
 		(on_board yes)
 		(dnp no)
-		(property "Reference" "U4"
+		(property "Reference" "IC4"
 			(at 129.286 62.992 0)
 			(effects
@@
 			(project ""
 				(path "/d6028aad-759f-4736-9818-30f0061d1d8d/721fd379-0889-4e74-8212-a23ae46bf4ef"
-					(reference "U4")
+					(reference "IC4")
 					(unit 2)
 				)
@@
 		(on_board yes)
 		(dnp no)
-		(property "Reference" "U4"
+		(property "Reference" "IC4"
 			(at 129.54 39.37 0)
 			(effects
@@
 			(project ""
 				(path "/d6028aad-759f-4736-9818-30f0061d1d8d/721fd379-0889-4e74-8212-a23ae46bf4ef"
-					(reference "U4")
+					(reference "IC4")
 					(unit 1)
 				)
@@
 		(on_board yes)
 		(dnp no)
-		(property "Reference" "U4"
+		(property "Reference" "IC4"
 			(at 129.794 112.268 0)
 			(effects
@@
 			(project ""
 				(path "/d6028aad-759f-4736-9818-30f0061d1d8d/721fd379-0889-4e74-8212-a23ae46bf4ef"
-					(reference "U4")
+					(reference "IC4")
 					(unit 4)
 				)
@@
 		(on_board yes)
 		(dnp no)
-		(property "Reference" "U4"
+		(property "Reference" "IC4"
 			(at 129.794 88.138 0)
 			(effects
@@
 			(project ""
 				(path "/d6028aad-759f-4736-9818-30f0061d1d8d/721fd379-0889-4e74-8212-a23ae46bf4ef"
-					(reference "U4")
+					(reference "IC4")
 					(unit 3)
 				)

Commit message: updates to banana pcb
Parts:
- added D1, D2, D3, D4: D_Zener, Diode_SMD:D_0805_2012Metric, symbol Device:D_Zener
- added Q1, Q2, Q3, Q4: 2N7002, Package_TO_SOT_SMD:SOT-23, symbol Transistor_FET:2N7002
Connections:
- net CV1: now also D1.1 (K)
- net CV2: now also D2.1 (K)
- net CV3: now also D3.1 (K)
- net CV4: now also D4.1 (K)
- net GND: now also Q1.2 (S), Q2.2 (S), Q3.2 (S), Q4.2 (S)
- new net: D2.2 (A), Q2.3 (D)
- new net: D4.2 (A), Q4.3 (D)
- new net: D3.2 (A), Q3.3 (D)
- new net: D1.2 (A), Q1.3 (D)
- new net CLAMP_EN: Q1.1 (G), Q2.1 (G), Q3.1 (G), Q4.1 (G)
Other:
- moved on the sheet: C19, IC4E

Commit message: banana updates
Connections:
- net +5V renamed +10V
Changed lines of the file:
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@@
-	)
-	(symbol
-		(lib_id "power:+5V")
-		(at 123.19 130.81 0)
-		(unit 1)
-		(exclude_from_sim no)
-		(in_bom yes)
-		(on_board yes)
-		(dnp no)
-		(property "Reference" "#PWR055"
-			(at 123.19 134.62 0)
-			(effects
-				(font
-					(size 1.27 1.27)
-				)
-				(hide yes)
-			)
-		)
-		(property "Value" "+5V"
-			(at 123.19 127 0)
-			(effects
-				(font
-					(size 1.27 1.27)
-				)
-			)
-		)
-		(property "Footprint" ""
-			(at 123.19 130.81 0)
-			(effects
-				(font
-					(size 1.27 1.27)
-				)
-				(hide yes)
-			)
-		)
-		(property "Datasheet" ""
-			(at 123.19 130.81 0)
-			(effects
-				(font
-					(size 1.27 1.27)
-				)
-				(hide yes)
-			)
-		)
-		(property "Description" "Power symbol creates a global label with name \"+5V\""
-			(at 123.19 130.81 0)
-			(effects
-				(font
-					(size 1.27 1.27)
-				)
-				(hide yes)
-			)
-		)
-		(pin "1"
-		)
-		(instances
-			(project "cvocd_banana"
-				(path "/d6028aad-759f-4736-9818-30f0061d1d8d/721fd379-0889-4e74-8212-a23ae46bf4ef"
-					(reference "#PWR055")
-					(unit 1)
-				)
-			)
-		)
 	)
 	(symbol
@@
 					(unit 1)
 				)
+			)
+		)
+	)
+	(symbol
+		(lib_id "power:+10V")
+		(at 123.19 130.81 0)
+		(unit 1)
+		(exclude_from_sim no)
+		(in_bom yes)
+		(on_board yes)
+		(dnp no)
+		(property "Reference" "#PWR055"
+			(at 123.19 134.62 0)
+			(effects
+				(font
+					(size 1.27 1.27)
+				)
+				(hide yes)
+			)
+		)
+		(property "Value" "+10V"
+			(at 122.936 127 0)
+			(effects
+				(font
+					(size 1.27 1.27)
+				)
+			)
+		)
+		(property "Footprint" ""
+			(at 123.19 130.81 0)
+			(effects
+				(font
+					(size 1.27 1.27)
+				)
+				(hide yes)
+			)
+		)
+		(property "Datasheet" ""
+			(at 123.19 130.81 0)
+			(effects
+				(font
+					(size 1.27 1.27)
+				)
+				(hide yes)
+			)
+		)
+		(property "Description" "Power symbol creates a global label with name \"+10V\""
+			(at 123.19 130.81 0)
+			(effects
+				(font
+					(size 1.27 1.27)
+				)
+				(hide yes)
+			)
+		)
+		(pin "1"
+		)
+		(instances
+			(project "cvocd_banana"
+				(path "/d6028aad-759f-4736-9818-30f0061d1d8d/721fd379-0889-4e74-8212-a23ae46bf4ef"
+					(reference "#PWR055")
+					(unit 1)
+				)

Commit message: banana pcb main v2
Parts:
- D1, D2, D3, D4: value D_Zener -> 5V1
Changed lines of the file:
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@@
 		)
 		(property "Value" "LM324"
-			(at 130.81 31.75 0)
-			(effects
-				(font
-					(size 1.27 1.27)
-				)
-				(hide yes)
+			(at 128.524 45.72 0)
+			(effects
+				(font
+					(size 1.27 1.27)
+				)
 			)
 		)
@@
 		(dnp no)
 		(property "Reference" "Q2"
-			(at 105.156 62.484 90)
+			(at 102.108 67.31 90)
 			(effects
 				(font
@@
 		)
 		(property "Value" "2N7002"
-			(at 100.33 57.15 90)
-			(effects
-				(font
-					(size 1.27 1.27)
-				)
-				(hide yes)
+			(at 104.648 69.088 90)
+			(effects
+				(font
+					(size 1.27 1.27)
+				)
 			)
 		)
@@
 		(dnp no)
 		(property "Reference" "Q4"
-			(at 105.156 110.744 90)
+			(at 102.362 115.57 90)
 			(effects
 				(font
@@
 		)
 		(property "Value" "2N7002"
-			(at 100.33 105.41 90)
-			(effects
-				(font
-					(size 1.27 1.27)
-				)
-				(hide yes)
+			(at 104.648 117.348 90)
+			(effects
+				(font
+					(size 1.27 1.27)
+				)
 			)
 		)
@@
 			)
 		)
-		(property "Value" "D_Zener"
-			(at 88.9 81.28 0)
-			(effects
-				(font
-					(size 1.27 1.27)
-				)
-				(hide yes)
+		(property "Value" "5V1"
+			(at 89.408 89.408 0)
+			(effects
+				(font
+					(size 1.27 1.27)
+				)
 			)
 		)
@@
 		(dnp no)
 		(property "Reference" "C19"
-			(at 128.27 128.778 90)
+			(at 129.286 135.382 90)
 			(effects
 				(font
@@
 		)
 		(property "Value" "100n"
-			(at 128.524 135.382 90)
+			(at 129.794 137.16 90)
 			(effects
 				(font
@@
 		(dnp no)
 		(property "Reference" "Q3"
-			(at 105.156 86.614 90)
+			(at 102.108 91.694 90)
 			(effects
 				(font
@@
 		)
 		(property "Value" "2N7002"
-			(at 100.33 81.28 90)
-			(effects
-				(font
-					(size 1.27 1.27)
-				)
-				(hide yes)
+			(at 104.648 93.472 90)
+			(effects
+				(font
+					(size 1.27 1.27)
+				)
 			)
 		)
@@
 			)
 		)
-		(property "Value" "D_Zener"
-			(at 88.9 33.02 0)
-			(effects
-				(font
-					(size 1.27 1.27)
-				)
-				(hide yes)
+		(property "Value" "5V1"
+			(at 89.408 41.148 0)
+			(effects
+				(font
+					(size 1.27 1.27)
+				)
 			)
 		)
@@
 		(dnp no)
 		(property "Reference" "Q1"
-			(at 105.156 38.354 90)
+			(at 102.108 43.18 90)
 			(effects
 				(font
@@
 		)
 		(property "Value" "2N7002"
-			(at 100.33 33.02 90)
-			(effects
-				(font
-					(size 1.27 1.27)
-				)
-				(hide yes)
+			(at 104.648 44.958 90)
+			(effects
+				(font
+					(size 1.27 1.27)
+				)
 			)
 		)
@@
 			)
 		)
-		(property "Value" "D_Zener"
-			(at 88.9 105.41 0)
-			(effects
-				(font
-					(size 1.27 1.27)
-				)
-				(hide yes)
+		(property "Value" "5V1"
+			(at 89.408 113.538 0)
+			(effects
+				(font
+					(size 1.27 1.27)
+				)
 			)
 		)
@@
 			)
 		)
-		(property "Value" "D_Zener"
-			(at 88.9 57.15 0)
-			(effects
-				(font
-					(size 1.27 1.27)
-				)
-				(hide yes)
-			)
-		)
+		(property "Value" "5V1"
+			(at 89.408 65.278 0)
+			(effects
+				(font
+					(size 1.27 1.27)
+				)
+			)
+		)
