File: cvocd_banana/cvocd_banana.kicad_sch (KiCad schematic)
At the start: 0 parts

Commit message: banana updates
Other:
- note added: "1- Added lower mounting hole and moved led/button solder points 2- Change orientation of limit switch 3- input for 5v reg comes from dc input not 10v 4- LED buffer amp powered from 10V not 5V 5- AP3012 boost reg used"
Changed lines of the file:
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@@
 	(generator_version "8.0")
 	(paper "A4")
+	(text "1- Added lower mounting hole and moved led/button solder points\n2- Change orientation of limit switch\n3- input for 5v reg comes from dc input not 10v\n4- LED buffer amp powered from 10V not 5V\n5- AP3012 boost reg used\n\n\n"
+		(exclude_from_sim no)
+		(at 44.958 30.734 0)
+		(effects
+			(font
+				(size 3.81 3.81)
+				(thickness 0.4763)
+			)
+			(justify left)
+		)
+	)
 	(sheet
 		(at 119.38 96.52)

Commit message: banana pcb main v2
Other:
- note removed: "1- Added lower mounting hole and moved led/button solder points 2- Change orientation of limit switch 3- input for 5v reg comes from dc input not 10v 4- LED buffer amp powered from 10V not 5V 5- AP3012 boost reg used"
Changed lines of the file:
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@@
 	(generator_version "8.0")
 	(paper "A4")
-	(text "1- Added lower mounting hole and moved led/button solder points\n2- Change orientation of limit switch\n3- input for 5v reg comes from dc input not 10v\n4- LED buffer amp powered from 10V not 5V\n5- AP3012 boost reg used\n\n\n"
+	(text_box "22/4/26\n1- Added lower mounting hole and moved led/button solder points\n2- Change orientation of limit switch\n3- input for 5v reg comes from dc input not 10v\n4- LED buffer amp powered from 10V not 5V\n5- AP3012 boost reg used"
 		(exclude_from_sim no)
-		(at 44.958 30.734 0)
+		(at 179.705 64.135 0)
+		(size 95.885 28.575)
+		(stroke
+			(width 0)
+			(type default)
+		)
+		(fill
+			(type none)
+		)
 		(effects
 			(font
-				(size 3.81 3.81)
-				(thickness 0.4763)
+				(size 2.032 2.032)
 			)
-			(justify left)
+			(justify left top)
 		)
 	)
 	(sheet
-		(at 119.38 96.52)
-		(size 12.7 5.08)
+		(at 32.385 32.385)
+		(size 12.7 3.81)
 		(fields_autoplaced yes)
 		(stroke
@@
 		)
 		(property "Sheetname" "gate_out"
-			(at 119.38 95.8084 0)
+			(at 32.385 31.6734 0)
 			(effects
 				(font
@@
 		)
 		(property "Sheetfile" "gate_out.kicad_sch"
-			(at 119.38 102.1846 0)
+			(at 32.385 36.7796 0)
 			(effects
 				(font
@@
 	)
 	(sheet
-		(at 121.92 109.22)
-		(size 12.7 5.08)
+		(at 32.385 43.18)
+		(size 12.7 3.81)
 		(fields_autoplaced yes)
 		(stroke
@@
 		)
 		(property "Sheetname" "cv_out"
-			(at 121.92 108.5084 0)
+			(at 32.385 42.4684 0)
 			(effects
 				(font
@@
 		)
 		(property "Sheetfile" "cv_out.kicad_sch"
-			(at 121.92 114.8846 0)
+			(at 32.385 47.5746 0)
 			(effects
 				(font
@@
 	)
 	(sheet
-		(at 121.92 127)
+		(at 32.385 54.61)
 		(size 12.7 3.81)
 		(fields_autoplaced yes)
@@
 		)
 		(property "Sheetname" "inputs"
-			(at 121.92 126.2884 0)
+			(at 32.385 53.8984 0)
 			(effects
 				(font
@@
 		)
 		(property "Sheetfile" "inputs.kicad_sch"
-			(at 121.92 131.3946 0)
+			(at 32.385 59.0046 0)
 			(effects
 				(font
