File: cvocd_banana/gate_out.kicad_sch (KiCad schematic)
At the start: 70 parts, among them U1 4504, U2 4504, U3 4504

Commit message: ASD
Parts:
- renumbered U1 to IC1, U2 to IC2, U3 to IC3, R13 to R11, R11 to R12, R12 to R13, R20 to R19, R3 to R2, R19 to R20, R23 to R22, R22 to R23, R5 to R3, R6 to R5, R7 to R6, R2 to R7, XG2 to XG1, XG9 to XG10, XG10 to XG11, XG11 to XG12, XG3 to XG2, XG4 to XG3, XG1 to XG4, XG8 to XG5, XG5 to XG6, XG6 to XG7, XG7 to XG8, XG12 to XG9

Commit message: REV1
Parts:
- renumbered XG11 to GATE10X1, XG12 to GATE11X1, XG9 to GATE12X1, XG4 to GATE1X1, XG1 to GATE2X1, XG2 to GATE3X1, XG3 to GATE4X1, XG6 to GATE5X1, XG7 to GATE6X1, XG8 to GATE7X1, XG5 to GATE8X1, XG10 to GATE9X1
Changed lines of the file:
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@@
 		(on_board yes)
 		(dnp no)
-		(property "Reference" "XG2"
+		(property "Reference" "GATE3X1"
 			(at 313.182 54.61 0)
 			(effects
@@
 			(project "cvocd_banana"
 				(path "/d6028aad-759f-4736-9818-30f0061d1d8d/53ea022f-21ec-467d-a620-575d4d777832"
-					(reference "XG2")
+					(reference "GATE3X1")
 					(unit 1)
 				)
@@
 		(on_board yes)
 		(dnp no)
-		(property "Reference" "XG6"
+		(property "Reference" "GATE5X1"
 			(at 311.912 135.89 0)
 			(effects
@@
 			(project "cvocd_banana"
 				(path "/d6028aad-759f-4736-9818-30f0061d1d8d/53ea022f-21ec-467d-a620-575d4d777832"
-					(reference "XG6")
+					(reference "GATE5X1")
 					(unit 1)
 				)
@@
 		(on_board yes)
 		(dnp no)
-		(property "Reference" "XG9"
+		(property "Reference" "GATE12X1"
 			(at 310.642 196.85 0)
 			(effects
@@
 			(project "cvocd_banana"
 				(path "/d6028aad-759f-4736-9818-30f0061d1d8d/53ea022f-21ec-467d-a620-575d4d777832"
-					(reference "XG9")
+					(reference "GATE12X1")
 					(unit 1)
 				)
@@
 		(on_board yes)
 		(dnp no)
-		(property "Reference" "XG8"
+		(property "Reference" "GATE7X1"
 			(at 311.912 146.05 0)
 			(effects
@@
 			(project "cvocd_banana"
 				(path "/d6028aad-759f-4736-9818-30f0061d1d8d/53ea022f-21ec-467d-a620-575d4d777832"
-					(reference "XG8")
+					(reference "GATE7X1")
 					(unit 1)
 				)
@@
 		(on_board yes)
 		(dnp no)
-		(property "Reference" "XG5"
+		(property "Reference" "GATE8X1"
 			(at 311.912 120.65 0)
 			(effects
@@
 			(project "cvocd_banana"
 				(path "/d6028aad-759f-4736-9818-30f0061d1d8d/53ea022f-21ec-467d-a620-575d4d777832"
-					(reference "XG5")
+					(reference "GATE8X1")
 					(unit 1)
 				)
@@
 		(on_board yes)
 		(dnp no)
-		(property "Reference" "XG1"
+		(property "Reference" "GATE2X1"
 			(at 313.182 49.53 0)
 			(effects
@@
 			(project "cvocd_banana"
 				(path "/d6028aad-759f-4736-9818-30f0061d1d8d/53ea022f-21ec-467d-a620-575d4d777832"
-					(reference "XG1")
+					(reference "GATE2X1")
 					(unit 1)
 				)
@@
 		(on_board yes)
 		(dnp no)
-		(property "Reference" "XG4"
+		(property "Reference" "GATE1X1"
 			(at 313.182 74.93 0)
 			(effects
@@
 			(project ""
 				(path "/d6028aad-759f-4736-9818-30f0061d1d8d/53ea022f-21ec-467d-a620-575d4d777832"
-					(reference "XG4")
+					(reference "GATE1X1")
 					(unit 1)
 				)
@@
 		(on_board yes)
 		(dnp no)
-		(property "Reference" "XG11"
+		(property "Reference" "GATE10X1"
 			(at 310.642 217.17 0)
 			(effects
@@
 			(project "cvocd_banana"
 				(path "/d6028aad-759f-4736-9818-30f0061d1d8d/53ea022f-21ec-467d-a620-575d4d777832"
-					(reference "XG11")
+					(reference "GATE10X1")
 					(unit 1)
 				)
@@
 		(on_board yes)
 		(dnp no)
-		(property "Reference" "XG10"
+		(property "Reference" "GATE9X1"
 			(at 310.642 212.09 0)
 			(effects
@@
 			(project "cvocd_banana"
 				(path "/d6028aad-759f-4736-9818-30f0061d1d8d/53ea022f-21ec-467d-a620-575d4d777832"
-					(reference "XG10")
+					(reference "GATE9X1")
 					(unit 1)
 				)
@@
 		(on_board yes)
 		(dnp no)
-		(property "Reference" "XG12"
+		(property "Reference" "GATE11X1"
 			(at 310.642 222.25 0)
 			(effects
@@
 			(project "cvocd_banana"
 				(path "/d6028aad-759f-4736-9818-30f0061d1d8d/53ea022f-21ec-467d-a620-575d4d777832"
-					(reference "XG12")
+					(reference "GATE11X1")
 					(unit 1)
 				)
@@
 		(on_board yes)
 		(dnp no)
-		(property "Reference" "XG7"
+		(property "Reference" "GATE6X1"
 			(at 311.912 140.97 0)
 			(effects
@@
 			(project "cvocd_banana"
 				(path "/d6028aad-759f-4736-9818-30f0061d1d8d/53ea022f-21ec-467d-a620-575d4d777832"
-					(reference "XG7")
+					(reference "GATE6X1")
 					(unit 1)
 				)
@@
 		(on_board yes)
 		(dnp no)
-		(property "Reference" "XG3"
+		(property "Reference" "GATE4X1"
 			(at 313.182 59.69 0)
 			(effects
@@
 			(project "cvocd_banana"
 				(path "/d6028aad-759f-4736-9818-30f0061d1d8d/53ea022f-21ec-467d-a620-575d4d777832"
-					(reference "XG3")
+					(reference "GATE4X1")
 					(unit 1)
 				)

Commit message: banana pcb main v2
Parts:
- C10, C11, C12, C15, C16, C17, C18, C3, C4, C5, C6, C9: value C -> 10n
Changed lines of the file:
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@@
 		(dnp no)
 		(property "Reference" "C11"
-			(at 283.972 151.384 0)
+			(at 282.956 149.86 0)
 			(effects
 				(font
@@
 			)
 		)
-		(property "Value" "C"
-			(at 285.242 155.702 0)
+		(property "Value" "10n"
+			(at 282.956 151.638 0)
 			(effects
 				(font
@@
 		(dnp no)
 		(property "Reference" "C5"
-			(at 285.242 80.264 0)
+			(at 285.496 78.74 0)
 			(effects
 				(font
@@
 			)
 		)
-		(property "Value" "C"
-			(at 286.512 84.582 0)
+		(property "Value" "10n"
+			(at 284.48 80.518 0)
 			(effects
 				(font
@@
 		(dnp no)
 		(property "Reference" "C9"
-			(at 273.812 151.384 0)
+			(at 273.812 149.86 0)
 			(effects
 				(font
@@
 			)
 		)
-		(property "Value" "C"
-			(at 275.082 155.702 0)
+		(property "Value" "10n"
+			(at 272.796 151.638 0)
 			(effects
 				(font
@@
 		(dnp no)
 		(property "Reference" "C18"
-			(at 287.782 227.584 0)
+			(at 286.766 226.06 0)
 			(effects
 				(font
@@
 			)
 		)
-		(property "Value" "C"
-			(at 289.052 231.902 0)
+		(property "Value" "10n"
+			(at 287.02 227.838 0)
 			(effects
 				(font
@@
 		(dnp no)
 		(property "Reference" "C15"
-			(at 272.542 227.584 0)
+			(at 271.526 226.06 0)
 			(effects
 				(font
@@
 			)
 		)
-		(property "Value" "C"
-			(at 273.812 231.902 0)
+		(property "Value" "10n"
+			(at 271.526 227.838 0)
 			(effects
 				(font
@@
 		(dnp no)
 		(property "Reference" "C4"
-			(at 280.162 80.264 0)
+			(at 280.416 78.74 0)
 			(effects
 				(font
@@
 			)
 		)
-		(property "Value" "C"
-			(at 281.432 84.582 0)
+		(property "Value" "10n"
+			(at 279.4 80.518 0)
 			(effects
 				(font
@@
 		(dnp no)
 		(property "Reference" "C6"
-			(at 290.322 80.264 0)
+			(at 290.576 78.74 0)
 			(effects
 				(font
@@
 			)
 		)
-		(property "Value" "C"
-			(at 291.592 84.582 0)
+		(property "Value" "10n"
+			(at 289.56 80.518 0)
 			(effects
 				(font
@@
 		(dnp no)
 		(property "Reference" "C17"
-			(at 282.702 227.584 0)
+			(at 281.686 226.06 0)
 			(effects
 				(font
@@
 			)
 		)
-		(property "Value" "C"
-			(at 283.972 231.902 0)
+		(property "Value" "10n"
+			(at 281.94 227.838 0)
 			(effects
 				(font
@@
 		(dnp no)
 		(property "Reference" "C3"
-			(at 275.082 80.264 0)
+			(at 274.32 78.74 0)
 			(effects
 				(font
@@
 			)
 		)
-		(property "Value" "C"
-			(at 276.352 84.582 0)
+		(property "Value" "10n"
+			(at 274.32 80.518 0)
 			(effects
 				(font
@@
 		(dnp no)
 		(property "Reference" "C16"
-			(at 277.622 227.584 0)
+			(at 276.606 226.06 0)
 			(effects
 				(font
@@
 			)
 		)
-		(property "Value" "C"
-			(at 278.892 231.902 0)
+		(property "Value" "10n"
+			(at 276.86 227.838 0)
 			(effects
 				(font
@@
 		(dnp no)
 		(property "Reference" "C10"
-			(at 278.892 151.384 0)
+			(at 277.876 149.86 0)
 			(effects
 				(font
@@
 			)
 		)
-		(property "Value" "C"
-			(at 280.162 155.702 0)
+		(property "Value" "10n"
+			(at 277.876 151.638 0)
 			(effects
 				(font
@@
 		(dnp no)
 		(property "Reference" "C12"
-			(at 289.052 151.384 0)
+			(at 288.036 149.86 0)
 			(effects
 				(font
@@
 			)
 		)
-		(property "Value" "C"
-			(at 290.322 155.702 0)
+		(property "Value" "10n"
+			(at 288.036 151.638 0)
 			(effects
 				(font
