File: cvocd_banana/inputs.kicad_sch (KiCad schematic)
At the start: 64 parts, among them SW1 SW_SP3T, SW2 SW_SP3T, SW3 SW_SP3T, U5 MC34063AD, U6 LM317L_SOT-89, U7 AMS1117

Commit message: ASD
Parts:
- renumbered U5 to IC5, U6 to IC6, U7 to IC7
Changed lines of the file:
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@@
 		(on_board yes)
 		(dnp no)
-		(property "Reference" "U5"
+		(property "Reference" "IC5"
 			(at 182.372 82.55 0)
 			(effects
@@
 			(project ""
 				(path "/d6028aad-759f-4736-9818-30f0061d1d8d/a7087e78-201a-4bde-9ba0-5717116ba4d1"
-					(reference "U5")
+					(reference "IC5")
 					(unit 1)
 				)
@@
 		(on_board yes)
 		(dnp no)
-		(property "Reference" "U6"
+		(property "Reference" "IC6"
 			(at 161.036 123.444 0)
 			(effects
@@
 			(project ""
 				(path "/d6028aad-759f-4736-9818-30f0061d1d8d/a7087e78-201a-4bde-9ba0-5717116ba4d1"
-					(reference "U6")
+					(reference "IC6")
 					(unit 1)
 				)
@@
 		(on_board yes)
 		(dnp no)
-		(property "Reference" "U7"
+		(property "Reference" "IC7"
 			(at 215.646 123.444 0)
 			(effects
@@
 			(project ""
 				(path "/d6028aad-759f-4736-9818-30f0061d1d8d/a7087e78-201a-4bde-9ba0-5717116ba4d1"
-					(reference "U7")
-					(unit 1)
-				)
+					(reference "IC7")
+					(unit 1)
+				)

Commit message: REV1
Parts:
- added GND4, POWER3, POWER4, POWER5: Conn_01x01, Jason_Kicad:WireToBoardCVOCD, symbol Connector_Generic:Conn_01x01
Connections:
- net +10V: now also POWER4.1 (Pin_1)
- net +15V: now also POWER3.1 (Pin_1)
- net +5V: now also POWER5.1 (Pin_1)
- net GND: now also GND4.1 (Pin_1)
Other:
- moved on the sheet: MIDI1, MIDI2, XMIDI1, XMIDI2

Commit message: updates to banana pcb
Parts:
- added R42: R, Resistor_SMD:R_0805_2012Metric, symbol Device:R
- added SW4: SW_SPDT, Jason_Kicad:Slide_1P2T_Rev_Mnt_CLSB12B01, symbol Switch:SW_SPDT
- SW1, SW2, SW3: footprint Jason_Kicad:Slide_SW_Rev_Mnt_CLSB13B01 -> Jason_Kicad:Slide_1P3T_Rev_Mnt_CLSB13B01
- renumbered D1 to D5, D2 to D6, D3 to D7, D4 to D8, D5 to D9
Connections:
- net +15V: now also SW1.4, SW2.4, SW3.4; no longer SW1.1, SW2.1, SW3.1
- net +5V: now also R42.1
- net GND: now also SW4.1 (A)
- new net CLAMP_EN: R42.2, SW4.2 (B)
- no-connect marks 3 -> 4

Commit message: banana updates
Parts:
- removed C21: C, Capacitor_SMD:C_0805_2012Metric, symbol Device:C
- removed C22: C_Polarized, Capacitor_SMD:CP_Elec_6.3x5.8, symbol Device:C_Polarized
- removed IC5: MC34063AD, Package_SO:SOIC-8_3.9x4.9mm_P1.27mm, symbol Regulator_Switching:MC34063AD
- removed R38, R39: R, Resistor_SMD:R_0805_2012Metric, symbol Device:R
- added C24, C25: C, Capacitor_SMD:C_1210_3225Metric_Pad1.33x2.70mm_HandSolder, symbol Device:C
- added IC6: AP3012, Package_TO_SOT_SMD:SOT-23-5, symbol Regulator_Switching:AP3012
- C22: renamed from C29; footprint Capacitor_SMD:CP_Elec_6.3x5.8 -> Capacitor_Tantalum_SMD:CP_EIA-6032-28_Kemet-C
- C23: footprint Capacitor_SMD:CP_Elec_6.3x5.8 -> Capacitor_Tantalum_SMD:CP_EIA-6032-28_Kemet-C
- C26: renamed from C20; footprint Capacitor_SMD:CP_Elec_6.3x5.8 -> Capacitor_Tantalum_SMD:CP_EIA-6032-28_Kemet-C
- C29: renamed from C26; footprint Capacitor_SMD:CP_Elec_6.3x5.8 -> Capacitor_Tantalum_SMD:CP_EIA-6032-28_Kemet-C
- L1: footprint Inductor_SMD:L_10.4x10.4_H4.8 -> Inductor_SMD:L_Taiyo-Yuden_MD-4040
- R36: value R -> 22k
- R37: value R -> 2k
- R38: renamed from R40; value R -> 470
- R39: renamed from R41; value R -> 3K3
- renumbered C27 to C20, C28 to C21, C24 to C27, C25 to C28, IC7 to IC5, IC6 to IC7, R42 to R40
Connections:
- net +10V: no longer C20.1, IC5.3 (VI)
- net GND: now also R37.2, SW4.3 (C), C24.2, C25.2, IC6.2 (GND); no longer SW4.1 (A)
- net at D6.1 (K), L2.1: now also R36.1, C25.1
- net at C26.1, D5.1 (K): now also C20.1, IC5.3 (VI), L1.1, C24.1, IC6.4 (~{SHDN}), IC6.5 (IN); no longer R36.1
- net at D6.2 (A), L1.2: now also IC6.1 (SW)
- net at R37.1: now also R36.2, IC6.3 (FB)
Other:
- moved on the sheet: C20, C21, C22, C23, C27, C28, C29, IC5, IC7, L2, R38, R39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

Commit message: banana pcb main v2
Parts:
- C20, C21, C27, C28: value C -> 100n
- C22: value C_Polarized -> 100u; footprint Capacitor_Tantalum_SMD:CP_EIA-6032-28_Kemet-C -> Capacitor_Tantalum_SMD:CP_EIA-7343-31_Kemet-D
- C23, C26, C29: value C_Polarized -> 100u/20; footprint Capacitor_Tantalum_SMD:CP_EIA-6032-28_Kemet-C -> Capacitor_Tantalum_SMD:CP_EIA-7343-31_Kemet-D
- C24, C25: value C -> 1u; footprint Capacitor_SMD:C_1210_3225Metric_Pad1.33x2.70mm_HandSolder -> Capacitor_SMD:C_0805_2012Metric
- D7, D8, D9: value D_Schottky -> MBR0520
- L1: value L -> TYS4012100M-10/10uH
- L2: value L -> CM322522-1R0KL/1uH
- R33, R34, R35: value R -> 1k
- R40: value R -> 10k
Changed lines of the file:
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@@
 			)
 		)
-		(property "Value" "L"
+		(property "Value" "TYS4012100M-10/10uH"
 			(at 214.63 64.77 90)
 			(effects
@@
 			)
 		)
-		(property "Value" "D_Schottky"
-			(at 49.276 157.48 0)
+		(property "Value" "MBR0520"
+			(at 45.974 159.258 0)
 			(effects
 				(font
 					(size 1.27 1.27)
 				)
-				(hide yes)
 			)
 		)
@@
 		(dnp no)
 		(property "Reference" "C20"
-			(at 205.74 49.276 0)
+			(at 200.66 43.434 0)
 			(effects
 				(font
@@
 			)
 		)
-		(property "Value" "C"
-			(at 203.962 44.196 0)
+		(property "Value" "100n"
+			(at 200.66 44.958 0)
 			(effects
 				(font
@@
 		(dnp no)
 		(property "Reference" "C29"
-			(at 199.644 134.366 0)
+			(at 199.644 128.27 0)
 			(effects
 				(font
@@
 			)
 		)
-		(property "Value" "C_Polarized"
-			(at 203.2 132.4609 0)
+		(property "Value" "100u/20"
+			(at 199.644 130.048 0)
 			(effects
 				(font
@@
 				)
 				(justify left)
-				(hide yes)
 			)
 		)
-		(property "Footprint" "Capacitor_Tantalum_SMD:CP_EIA-6032-28_Kemet-C"
+		(property "Footprint" "Capacitor_Tantalum_SMD:CP_EIA-7343-31_Kemet-D"
 			(at 200.3552 135.89 0)
 			(effects
@@
 		(dnp no)
 		(property "Reference" "C22"
-			(at 230.124 49.276 0)
+			(at 229.87 49.022 0)
 			(effects
 				(font
@@
 			)
 		)
-		(property "Value" "C_Polarized"
-			(at 233.68 47.3709 0)
+		(property "Value" "100u"
+			(at 229.87 50.8 0)
 			(effects
 				(font
@@
 				)
 				(justify left)
-				(hide yes)
 			)
 		)
-		(property "Footprint" "Capacitor_Tantalum_SMD:CP_EIA-6032-28_Kemet-C"
+		(property "Footprint" "Capacitor_Tantalum_SMD:CP_EIA-7343-31_Kemet-D"
 			(at 230.8352 50.8 0)
 			(effects
@@
 		(on_board yes)
 		(dnp no)
-		(fields_autoplaced yes)
 		(property "Reference" "R40"
-			(at 57.15 167.6399 0)
+			(at 55.88 167.64 0)
 			(effects
 				(font
@@
 			)
 		)
-		(property "Value" "R"
-			(at 57.15 170.1799 0)
+		(property "Value" "10k"
+			(at 55.88 169.418 0)
 			(effects
 				(font
@@
 		(dnp no)
 		(property "Reference" "C26"
-			(at 161.036 94.996 0)
+			(at 165.354 88.9 0)
 			(effects
 				(font
@@
 			)
 		)
-		(property "Value" "C_Polarized"
-			(at 168.91 93.0909 0)
+		(property "Value" "100u/20"
+			(at 165.354 90.678 0)
 			(effects
 				(font
@@
 				)
 				(justify left)
-				(hide yes)
 			)
 		)
-		(property "Footprint" "Capacitor_Tantalum_SMD:CP_EIA-6032-28_Kemet-C"
+		(property "Footprint" "Capacitor_Tantalum_SMD:CP_EIA-7343-31_Kemet-D"
 			(at 166.0652 96.52 0)
 			(effects
@@
 			)
 		)
-		(property "Value" "R"
+		(property "Value" "1k"
 			(at 101.854 34.29 90)
 			(effects
@@
 			)
 		)
-		(property "Value" "R"
+		(property "Value" "1k"
 			(at 101.854 43.18 90)
 			(effects
@@
 		(dnp no)
 		(property "Reference" "R38"
-			(at 187.706 132.08 90)
+			(at 183.134 132.08 90)
 			(effects
 				(font
@@
 		(dnp no)
 		(property "Reference" "R39"
-			(at 187.706 143.51 90)
+			(at 183.134 143.002 90)
 			(effects
 				(font
@@
 		(dnp no)
 		(property "Reference" "C28"
-			(at 193.04 134.366 0)
+			(at 188.976 128.27 0)
 			(effects
 				(font
@@
 			)
 		)
-		(property "Value" "C"
-			(at 191.262 129.286 0)
+		(property "Value" "100n"
+			(at 187.96 130.048 0)
 			(effects
 				(font
@@
 			)
 		)
-		(property "Value" "R"
+		(property "Value" "1k"
 			(at 101.854 25.4 90)
 			(effects
@@
 		(dnp no)
 		(property "Reference" "C27"
-			(at 165.1 134.366 0)
+			(at 161.036 128.27 0)
 			(effects
 				(font
@@
 			)
 		)
-		(property "Value" "C"
-			(at 163.322 129.286 0)
+		(property "Value" "100n"
+			(at 160.02 130.048 0)
 			(effects
 				(font
@@
 			)
 		)
-		(property "Value" "D_Schottky"
-			(at 49.276 114.3 0)
+		(property "Value" "MBR0520"
+			(at 45.974 116.332 0)
 			(effects
 				(font
 					(size 1.27 1.27)
 				)
-				(hide yes)
 			)
 		)
@@
 		(dnp no)
 		(property "Reference" "R37"
-			(at 241.046 92.456 90)
+			(at 236.728 92.456 90)
 			(effects
 				(font
@@
 		(dnp no)
 		(property "Reference" "R36"
-			(at 241.046 82.55 90)
+			(at 236.728 82.296 90)
 			(effects
 				(font
@@
 		(dnp no)
 		(property "Reference" "C24"
-			(at 198.12 91.186 0)
+			(at 193.04 85.09 0)
 			(effects
 				(font
@@
 			)
 		)
-		(property "Value" "C"
-			(at 196.342 86.106 0)
+		(property "Value" "1u"
+			(at 193.04 86.868 0)
 			(effects
 				(font
@@
 			)
 		)
-		(property "Footprint" "Capacitor_SMD:C_1210_3225Metric_Pad1.33x2.70mm_HandSolder"
+		(property "Footprint" "Capacitor_SMD:C_0805_2012Metric"
 			(at 199.0852 92.71 0)
 			(effects
@@
 			)
 		)
-		(property "Value" "D_Schottky"
-			(at 49.276 135.89 0)
+		(property "Value" "MBR0520"
+			(at 46.228 137.668 0)
 			(effects
 				(font
 					(size 1.27 1.27)
 				)
-				(hide yes)
 			)
 		)
@@
 		(dnp no)
 		(property "Reference" "C25"
-			(at 246.38 91.186 0)
+			(at 246.38 85.09 0)
 			(effects
 				(font
@@
 			)
 		)
-		(property "Value" "C"
-			(at 244.602 86.106 0)
+		(property "Value" "1u"
+			(at 246.38 86.868 0)
 			(effects
 				(font
@@
 			)
 		)
-		(property "Footprint" "Capacitor_SMD:C_1210_3225Metric_Pad1.33x2.70mm_HandSolder"
+		(property "Footprint" "Capacitor_SMD:C_0805_2012Metric"
 			(at 247.3452 92.71 0)
 			(effects
@@
 			)
 		)
-		(property "Value" "L"
+		(property "Value" "CM322522-1R0KL/1uH"
 			(at 255.27 74.93 90)
 			(effects
@@
 		(dnp no)
 		(property "Reference" "C21"
-			(at 223.52 49.276 0)
+			(at 218.44 49.022 0)
 			(effects
 				(font
@@
 			)
 		)
-		(property "Value" "C"
-			(at 221.742 44.196 0)
+		(property "Value" "100n"
+			(at 218.44 50.8 0)
 			(effects
 				(font
@@
 		(dnp no)
 		(property "Reference" "C23"
-			(at 256.286 88.646 0)
+			(at 260.604 82.042 0)
 			(effects
 				(font
@@
 			)
 		)
-		(property "Value" "C_Polarized"
-			(at 264.16 86.7409 0)
+		(property "Value" "100u/20"
+			(at 260.604 84.074 0)
 			(effects
 				(font
@@
 				)
 				(justify left)
-				(hide yes)
 			)
 		)
-		(property "Footprint" "Capacitor_Tantalum_SMD:CP_EIA-6032-28_Kemet-C"
+		(property "Footprint" "Capacitor_Tantalum_SMD:CP_EIA-7343-31_Kemet-D"
 			(at 261.3152 90.17 0)
 			(effects
